Commit message: updates to support 2 arms
- updated URDF

- updated JACO drivers

- updated gripper controller
*this needs a more elegant solution, the serial comm requires time between read/write and needs to be flushed before a transaction, this is just a temporary fix. It works but the update rate has to be reduced. Need to test multiprocessing queue implementation of the standalone serial driver with this when I get a chance.

File: vector_common/vector_description/urdf/linear_actuator/vector_linear_actuator.urdf.xacro (robot description, xacro)
@@ -52,20 +52,40 @@
             <dynamics damping="0.0" friction="0.0"/>
         </joint>
-        <link name="linear_actuator_link">
-			<visual>
-				<geometry>
-					<mesh filename="package://vector_description/meshes/linear_actuator/visual/linear_carraige.dae" />
-				</geometry>
-			</visual>
-			<collision>
-				<geometry>
-					<mesh filename="package://vector_description/meshes/linear_actuator/collision/linear_carraige_collision.STL" />
-				</geometry>
-			</collision>
-		    <inertial>
-			    <mass value="2e-06"/>
-			    <inertia ixx="1.1e-09" ixy="0" ixz="0" iyy="1.1e-09" iyz="0" izz="1.1e-09"/>
-		    </inertial>
-		</link>
+        <xacro:unless value="$(optenv VECTOR_HAS_TWO_KINOVA_ARMS false)">
+            <link name="linear_actuator_link">
+			    <visual>
+				    <geometry>
+					    <mesh filename="package://vector_description/meshes/linear_actuator/visual/linear_carraige.dae" />
+				    </geometry>
+			    </visual>
+			    <collision>
+				    <geometry>
+					    <mesh filename="package://vector_description/meshes/linear_actuator/collision/linear_carraige_collision.STL" />
+				    </geometry>
+			    </collision>
+		        <inertial>
+			        <mass value="2e-06"/>
+			        <inertia ixx="1.1e-09" ixy="0" ixz="0" iyy="1.1e-09" iyz="0" izz="1.1e-09"/>
+		        </inertial>
+		    </link>
+		</xacro:unless>
+        <xacro:if value="$(optenv VECTOR_HAS_TWO_KINOVA_ARMS false)">
+            <link name="linear_actuator_link">
+			    <visual>
+				    <geometry>
+					    <mesh filename="package://vector_description/meshes/linear_actuator/visual/linear_carraige_dual_front.dae" />
+				    </geometry>
+			    </visual>
+			    <collision>
+				    <geometry>
+					    <mesh filename="package://vector_description/meshes/linear_actuator/collision/linear_carraige_dual_front.STL" />
+				    </geometry>
+			    </collision>
+		        <inertial>
+			        <mass value="2e-06"/>
+			        <inertia ixx="1.1e-09" ixy="0" ixz="0" iyy="1.1e-09" iyz="0" izz="1.1e-09"/>
+		        </inertial>
+		    </link>
+		</xacro:if>
         <transmission name="linear_trans">
             <type>transmission_interface/SimpleTransmission</type>

File: vector_common/vector_description/urdf/vector.urdf.xacro (robot description, xacro)
@@ -49,9 +49,14 @@
     <xacro:if value="$(optenv VECTOR_HAS_KINOVA_ARM false)">
         <xacro:jaco_robot prefix="right_" parent="linear_actuator_link">
-            <origin xyz="0.06079866 0 0" rpy="${M_PI/2} 0 ${M_PI/2}"/>
+            <xacro:unless value="$(optenv VECTOR_HAS_TWO_KINOVA_ARMS false)">
+                <origin xyz="0.06079866 0 0" rpy="${M_PI/2} 0 ${M_PI/2}"/>
+            </xacro:unless>
+            <xacro:if value="$(optenv VECTOR_HAS_TWO_KINOVA_ARMS false)">
+                <origin xyz="0.06079866 -0.1319 0" rpy="${M_PI/2} 0 ${M_PI/2}"/>
+            </xacro:if>
         </xacro:jaco_robot>
         <xacro:if value="$(optenv VECTOR_HAS_TWO_KINOVA_ARMS false)">
             <xacro:jaco_robot prefix="left_" parent="linear_actuator_link">
-                <origin xyz="0.06079866 0 0" rpy="${M_PI/2} 0 ${M_PI/2}"/>
+                <origin xyz="0.06079866 0.1319 0" rpy="${M_PI/2} 0 ${M_PI/2}"/>
             </xacro:jaco_robot>
         </xacro:if>
@@ -61,5 +66,5 @@
             </xacro:robotiq_85_gripper>
             <xacro:if value="$(optenv VECTOR_HAS_TWO_ROBOTIQ_GRIPPERS false)">
-                <xacro:robotiq_85_gripper prefix="left_" parent="right_ee_link" >
+                <xacro:robotiq_85_gripper prefix="left_" parent="left_ee_link" >
                     <origin xyz="0 0 0" rpy="0 0 0"/>
                 </xacro:robotiq_85_gripper>

Commit message: Merge in changes to the URDF to make the robot stable in simulation and match kinova API. Also added in link for gripper and changes to allow for simulation teleop

File: vector_common/vector_description/urdf/linear_actuator/vector_linear_actuator.urdf.xacro (robot description, xacro)
@@ -40,6 +40,9 @@
 			</collision>
 		    <inertial>
-			    <mass value="2e-06"/>
-			    <inertia ixx="1.1e-09" ixy="0" ixz="0" iyy="1.1e-09" iyz="0" izz="1.1e-09"/>
+                <!--mass value="2e-06"/>
+                <inertia ixx="1.1e-09" ixy="0" ixz="0" iyy="1.1e-09" iyz="0" izz="1.1e-09"/-->
+                <mass value="5.098044" />
+                <origin xyz="0.0 0.0 0.5" rpy="0 0 0"/>
+                <inertia ixx="0.02"  ixy="0.0"  ixz="1.0" iyy="-0.03"  iyz="-0.02" izz="0.0" />
 		    </inertial>
 		</link>
@@ -65,6 +68,11 @@
 			    </collision>
 		        <inertial>
-			        <mass value="2e-06"/>
-			        <inertia ixx="1.1e-09" ixy="0" ixz="0" iyy="1.1e-09" iyz="0" izz="1.1e-09"/>
+                    <!--mass value="2e-06"/>
+                    <inertia ixx="1.1e-09" ixy="0" ixz="0" iyy="1.1e-09" iyz="0" izz="1.1e-09"/-->
+                    <mass value="0.217" />
+                    <origin xyz="0 -0.001 0" rpy="0 0 0"/>
+                    <inertia ixx="0.0" ixy="0.0"  ixz="1.0"
+                             iyy="0.0" iyz="0.0"
+                             izz="0.0" />
 		        </inertial>
 		    </link>

File: vector_common/vector_description/urdf/manipulation/jaco/jaco.urdf.xacro (robot description, xacro)
@@ -87,7 +87,9 @@
             <parent link="${prefix}shoulder_link" />
             <child link = "${prefix}upper_arm_link" />
-            <origin xyz="0 0 -0.11875" rpy="${M_PI/2} ${M_PI/2} 0" />
-            <axis xyz="0 0 1" />
-            <limit lower="-2.238" upper="2.238" effort="3000.5" velocity="0.314"/>
+            <!--ZERO CONFIG:<origin xyz="0 0 -0.11875" rpy="${M_PI/2} ${M_PI/2} 0" />-->
+            <origin xyz="0 0 -0.11875" rpy="${M_PI/2} ${-M_PI/2} 0" />
+            <axis xyz="0 0 1" />
+            <!--ZERO CONFIG:<limit lower="-2.238" upper="2.238" effort="3000.5" velocity="0.314"/>-->
+            <limit lower="${M_PI-2.238}" upper="${M_PI+2.238}" effort="3000.5" velocity="0.314"/>
             <dynamics damping="0.0" friction="0.0"/>
         </joint>
@@ -114,7 +116,9 @@
             <parent link="${prefix}upper_arm_link" />
             <child link = "${prefix}forearm_link" />
-            <origin xyz="0.41 0 0.00975" rpy=" 0 ${M_PI} ${M_PI}" />
-            <axis xyz="0 0 1" />
-            <limit lower="-2.809" upper="2.809" effort="1800.0" velocity="0.314"/>
+            <!--ZERO CONFIG:<origin xyz="0.41 0 0.00975" rpy=" 0 ${M_PI} ${M_PI}" />-->
+            <origin xyz="0.41 0 0.00975" rpy="0 ${M_PI} 0" />
+            <axis xyz="0 0 1" />
+            <!--ZERO CONFIG:<limit lower="-2.809" upper="2.809" effort="1800.0" velocity="0.314"/>-->
+            <limit lower="${M_PI-2.809}" upper="${M_PI+2.809}" effort="1800.0" velocity="0.314"/>
             <dynamics damping="0.0" friction="0.0"/>
         </joint>
@@ -221,6 +225,13 @@
         <joint name="${prefix}ee_fixed_joint" type="fixed">
             <parent link="${prefix}wrist_3_link" />
-            <child link = "${prefix}ee_link" />
+            <child link = "${prefix}ee_base" />
             <origin xyz="0 0 -0.09380704" rpy="${M_PI} ${M_PI/2} 0" /> <!--0.09380704156-->
+        </joint>
+        <link name="${prefix}ee_base"/>
+        <!-- Add in an EEF link for the center of the gripper -->
+        <joint name="${prefix}ee_gripper" type="fixed">
+            <parent link="${prefix}ee_base" />
+            <child link ="${prefix}ee_link" />
+            <origin xyz="0.13 0 0" />
         </joint>
         <link name="${prefix}ee_link"/>

File: vector_common/vector_description/urdf/vector.urdf.xacro (robot description, xacro)
@@ -40,5 +40,5 @@
             <robotBaseFrame>base_link</robotBaseFrame>
             <publishOdometryTf>0</publishOdometryTf>
-            <yaw_velocity_p_gain>10000.0</yaw_velocity_p_gain>
+            <yaw_velocity_p_gain>100.0</yaw_velocity_p_gain>
             <x_velocity_p_gain>10000.0</x_velocity_p_gain>
             <y_velocity_p_gain>10000.0</y_velocity_p_gain>
@@ -68,9 +68,9 @@
         </xacro:if>
         <xacro:if value="$(optenv VECTOR_HAS_ROBOTIQ_GRIPPER false)">
-            <xacro:robotiq_85_gripper prefix="right_" parent="right_ee_link" >
+            <xacro:robotiq_85_gripper prefix="right_" parent="right_ee_base" >
                 <origin xyz="0 0 0" rpy="0 0 0"/>
             </xacro:robotiq_85_gripper>
             <xacro:if value="$(optenv VECTOR_HAS_TWO_ROBOTIQ_GRIPPERS false)">
-                <xacro:robotiq_85_gripper prefix="left_" parent="left_ee_link" >
+                <xacro:robotiq_85_gripper prefix="left_" parent="left_ee_base" >
                     <origin xyz="0 0 0" rpy="0 0 0"/>
                 </xacro:robotiq_85_gripper>
