Commit message: changed 3d simulation plugin and added flag to increase base inertia when in simulation

File: vector_common/vector_description/urdf/vector.urdf.xacro (robot description, xacro)
@@ -33,5 +33,5 @@
           <robotNamespace>/</robotNamespace>
         </plugin>
-        <plugin name="object_controller" filename="libgazebo_ros_force_based_move.so">
+        <plugin name="object_controller" filename="libgazebo_ros_planar_move.so">
             <commandTopic>/vector/cmd_vel</commandTopic>
             <odometryTopic>/vector/feedback/wheel_odometry</odometryTopic>
@@ -40,7 +40,4 @@
             <robotBaseFrame>base_link</robotBaseFrame>
             <publishOdometryTf>0</publishOdometryTf>
-            <yaw_velocity_p_gain>100.0</yaw_velocity_p_gain>
-            <x_velocity_p_gain>10000.0</x_velocity_p_gain>
-            <y_velocity_p_gain>10000.0</y_velocity_p_gain>
         </plugin>
     </gazebo>

File: vector_common/vector_description/urdf/vector_components/vector_base.urdf.xacro (robot description, xacro)
@@ -37,10 +37,18 @@
         <link name="${name}_chassis_link">
 			<inertial>
-				<mass value="55.914402" />
-				<origin xyz="0 0 0" />
-				<inertia ixx="3.54"  ixy="0" ixz="0"
-                         iyx="0"  iyy="3.71" iyz="0"
-                         izx="0" izy="0" izz="2.53" />
-			</inertial>
+                <mass value="55.914402" />
+                <origin xyz="0 0 0" />
+                <xacro:unless value="$(arg simulation_urdf)">
+                    <inertia ixx="3.53"  ixy="0" ixz="0"
+                             iyx="0"  iyy="3.71" iyz="0"
+                             izx="0" izy="0" izz="2.53" />
+                </xacro:unless>
+                <!-- Set appropriate inertial values if in simulation -->
+                <xacro:if value="$(arg simulation_urdf)">
+                    <inertia ixx="3000"  ixy="0" ixz="0"
+                             iyx="3000"  iyy="3.71" iyz="0"
+                             izx="3000" izy="0" izz="2.53" />
+                </xacro:if>
+            </inertial>
             <collision>
 				<geometry>
