Commit message: major updates after integration
gazebo sim and moveit configuration also updated

File: vector_common/vector_description/urdf/accessories.urdf.xacro (robot description, xacro)
@@ -28,4 +28,24 @@
     <property name="M_PI" value="3.14159"/>
     <xacro:macro name="vector_accessories">
+        <link name="sic_imu_frame"/>
+        <joint name="sic_imu_joint" type="fixed">
+            <origin xyz="0.07475 0.07136 0.24556" rpy="${M_PI} 0 0" />
+            <parent link="$(optenv VECTOR_PARENT_LINK base_chassis_link)" />
+            <child link="sic_imu_frame" />
+        </joint>
+        <gazebo>
+            <plugin name="sic_imu_controller" filename="libhector_gazebo_ros_imu.so">
+                <alwaysOn>1</alwaysOn>
+                <updateRate>50.0</updateRate>
+                <bodyName>sic_imu_frame</bodyName>
+                <topicName>/vector/feedback/sic_imu</topicName>
+                <accelDrift>0.005 0.005 0.005</accelDrift>
+                <accelGaussianNoise>0.005 0.005 0.005</accelGaussianNoise>
+                <rateDrift>0.005 0.005 0.005 </rateDrift>
+                <rateGaussianNoise>0.005 0.005 0.005 </rateGaussianNoise>
+                <headingDrift>0.005</headingDrift>
+                <headingGaussianNoise>0.005</headingGaussianNoise>
+            </plugin>
+        </gazebo>
         <!-- CH Robotics UM7 Link-->
         <xacro:if value="$(optenv VECTOR_HAS_EXT_IMU false)">
@@ -37,5 +57,5 @@
             </joint>
             <gazebo>
-                <plugin name="imu_controller" filename="libhector_gazebo_ros_imu.so">
+                <plugin name="ext_imu_controller" filename="libhector_gazebo_ros_imu.so">
                     <alwaysOn>1</alwaysOn>
                     <updateRate>50.0</updateRate>
@@ -58,7 +78,7 @@
         </xacro:if>
         <!-- SICK LMS1XX Sensor -->
-        <xacro:if value="$(optenv VECTOR_HAS_SICK false)">
+        <xacro:if value="$(optenv VECTOR_HAS_SICK_TIM false)">
             <xacro:sick_lms1xx laser_prefix="base" parent="$(optenv VECTOR_PARENT_LINK base_chassis_link)">
-                <origin xyz="$(optenv SICK_LMS1XX_XYZ 0 0 1.0)" rpy="$(optenv SICK_LMS1XX_RPY 3.14159 0 0)" />
+                <origin xyz="$(optenv SICK_TIM_XYZ 0 0 1.0)" rpy="$(optenv SICK_TIM_RPY 3.14159 0 0)" />
             </xacro:sick_lms1xx>
         </xacro:if>

File: vector_common/vector_description/urdf/manipulation/jaco/jaco.urdf.xacro (robot description, xacro)
@@ -62,5 +62,5 @@
             <origin xyz="0 0 0.15675" rpy="${M_PI} 0 ${M_PI}" />
             <axis xyz="0 0 1" />
-            <limit effort="18.0" velocity="0.314"/>
+            <limit effort="1800.0" velocity="0.314"/>
             <dynamics damping="0.0" friction="0.0"/>
         </joint>
@@ -89,5 +89,5 @@
             <origin xyz="0 0 -0.11875" rpy="${M_PI/2} ${M_PI/2} 0" />
             <axis xyz="0 0 1" />
-            <limit lower="-2.238" upper="2.238" effort="30.5" velocity="0.314"/>
+            <limit lower="-2.238" upper="2.238" effort="3000.5" velocity="0.314"/>
             <dynamics damping="0.0" friction="0.0"/>
         </joint>
@@ -116,5 +116,5 @@
             <origin xyz="0.41 0 0.00975" rpy=" 0 ${M_PI} ${M_PI}" />
             <axis xyz="0 0 1" />
-            <limit lower="-2.809" upper="2.809" effort="18.0" velocity="0.314"/>
+            <limit lower="-2.809" upper="2.809" effort="1800.0" velocity="0.314"/>
             <dynamics damping="0.0" friction="0.0"/>
         </joint>
@@ -143,5 +143,5 @@
             <origin xyz="0.20725 0 0 " rpy="0 -${M_PI/2} 0" />
             <axis xyz="0 0 1" />
-            <limit effort="6.8" velocity="0.785"/>
+            <limit effort="600.8" velocity="0.785"/>
             <dynamics damping="0.0" friction="0.0"/>
         </joint>
@@ -170,5 +170,5 @@
             <origin xyz="0 0 -0.04275704" rpy="0 ${M_PI/3} ${M_PI}" />
             <axis xyz="0 0 1" />
-            <limit effort="6.8" velocity="0.785"/>
+            <limit effort="600.8" velocity="0.785"/>
             <dynamics damping="0.0" friction="0.0"/>
         </joint>
@@ -197,5 +197,5 @@
             <origin xyz="0 0 -0.08551408" rpy="0 -${M_PI/3} 0" />
             <axis xyz="0 0 1" />
-            <limit effort="6.8" velocity="0.785"/>
+            <limit effort="600.8" velocity="0.785"/>
             <dynamics damping="0.0" friction="0.0"/>
         </joint>

File: vector_common/vector_description/urdf/manipulation/robotiq/robotiq_85_gripper.transmission.xacro (robot description, xacro)
@@ -9,69 +9,40 @@
             <actuator name="${prefix}robotiq_85_left_knuckle_motor">
                 <mechanicalReduction>1</mechanicalReduction>
+                <hardwareInterface>PositionJointInterface</hardwareInterface>
             </actuator>
         </transmission>
-        <transmission name="${prefix}robotiq_85_right_knuckle_trans">
-            <type>transmission_interface/SimpleTransmission</type>
-            <joint name="${prefix}robotiq_85_right_knuckle_joint">
-                <hardwareInterface>PositionJointInterface</hardwareInterface>
-            </joint>
-            <actuator name="${prefix}robotiq_85_right_knuckle_motor">
-                <mechanicalReduction>1</mechanicalReduction>
-            </actuator>
-        </transmission>
-        <transmission name="${prefix}robotiq_85_left_inner_knuckle_trans">
-            <type>transmission_interface/SimpleTransmission</type>
-            <joint name="${prefix}robotiq_85_left_inner_knuckle_joint">
-                <hardwareInterface>PositionJointInterface</hardwareInterface>
-            </joint>
-            <actuator name="${prefix}robotiq_85_left_inner_knuckle_motor">
-                <mechanicalReduction>1</mechanicalReduction>
-            </actuator>
-        </transmission>
-        <transmission name="${prefix}robotiq_85_right_inner_knuckle_trans">
-            <type>transmission_interface/SimpleTransmission</type>
-            <joint name="${prefix}robotiq_85_right_inner_knuckle_joint">
-                <hardwareInterface>PositionJointInterface</hardwareInterface>
-            </joint>
-            <actuator name="${prefix}robotiq_85_right_inner_knuckle_motor">
-                <mechanicalReduction>1</mechanicalReduction>
-            </actuator>
-        </transmission>
-        <!--transmission name="${prefix}robotiq_85_right_finger_trans">
-            <type>transmission_interface/SimpleTransmission</type>
-            <joint name="${prefix}robotiq_85_right_finger_joint">
-                <hardwareInterface>PositionJointInterface</hardwareInterface>
-            </joint>
-            <actuator name="${prefix}robotiq_85_right_finger_motor">
-                <mechanicalReduction>1</mechanicalReduction>
-            </actuator>
-        </transmission-->
-        <!--transmission name="${prefix}robotiq_85_left_finger_trans">
-            <type>transmission_interface/SimpleTransmission</type>
-            <joint name="${prefix}robotiq_85_left_finger_joint">
-                <hardwareInterface>PositionJointInterface</hardwareInterface>
-            </joint>
-            <actuator name="${prefix}robotiq_85_left_finger_motor">
-                <mechanicalReduction>1</mechanicalReduction>
-            </actuator>
-        </transmission-->
-        <transmission name="${prefix}robotiq_85_left_finger_tip_trans">
-            <type>transmission_interface/SimpleTransmission</type>
-            <joint name="${prefix}robotiq_85_left_finger_tip_joint">
-                <hardwareInterface>PositionJointInterface</hardwareInterface>
-            </joint>
-            <actuator name="${prefix}robotiq_85_left_finger_tip_motor">
-                <mechanicalReduction>1</mechanicalReduction>
-            </actuator>
-        </transmission>
-        <transmission name="${prefix}robotiq_85_right_finger_tip_trans">
-            <type>transmission_interface/SimpleTransmission</type>
-            <joint name="${prefix}robotiq_85_right_finger_tip_joint">
-                <hardwareInterface>PositionJointInterface</hardwareInterface>
-            </joint>
-            <actuator name="${prefix}robotiq_85_right_finger_tip_motor">
-                <mechanicalReduction>1</mechanicalReduction>
-            </actuator>
-        </transmission>
+        <gazebo>
+                <!-- loading plugin: mimic joints works in gazebo now -->
+            <plugin filename="libroboticsgroup_gazebo_mimic_joint_plugin.so" name="${prefix}mimic_robotiq_85_1">
+                <joint>${prefix}robotiq_85_left_knuckle_joint</joint>
+                <mimicJoint>${prefix}robotiq_85_right_knuckle_joint</mimicJoint>
+                <!--multiplier>1.0</multiplier>
+                <offset>0.0</offset-->
+            </plugin>
+            <plugin filename="libroboticsgroup_gazebo_mimic_joint_plugin.so" name="${prefix}mimic_robotiq_85_2">
+                <joint>${prefix}robotiq_85_left_knuckle_joint</joint>
+                <mimicJoint>${prefix}robotiq_85_left_inner_knuckle_joint</mimicJoint>
+                <!--multiplier>1.0</multiplier>
+                <offset>0.0</offset-->
+            </plugin>
+            <plugin filename="libroboticsgroup_gazebo_mimic_joint_plugin.so" name="${prefix}mimic_robotiq_85_3">
+                <joint>${prefix}robotiq_85_left_knuckle_joint</joint>
+                <mimicJoint>${prefix}robotiq_85_right_inner_knuckle_joint</mimicJoint>
+                <!--multiplier>1.0</multiplier>
+                <offset>0.0</offset-->
+            </plugin>
+            <plugin filename="libroboticsgroup_gazebo_mimic_joint_plugin.so" name="${prefix}mimic_robotiq_85_4">
+                <joint>${prefix}robotiq_85_left_knuckle_joint</joint>
+                <mimicJoint>${prefix}robotiq_85_left_finger_tip_joint</mimicJoint>
+                <multiplier>-1.0</multiplier>
+                <offset>0.0</offset>
+            </plugin>
+            <plugin filename="libroboticsgroup_gazebo_mimic_joint_plugin.so" name="${prefix}mimic_robotiq_85_5">
+                <joint>${prefix}robotiq_85_left_knuckle_joint</joint>
+                <mimicJoint>${prefix}robotiq_85_right_finger_tip_joint</mimicJoint>
+                <multiplier>-1.0</multiplier>
+                <offset>0.0</offset>
+            </plugin>
+        </gazebo>
     </xacro:macro>
 </robot>

File: vector_common/vector_description/urdf/manipulation/robotiq/robotiq_85_gripper.urdf.xacro (robot description, xacro)
@@ -35,21 +35,12 @@
             <limit lower="0.0" upper="0.804" velocity="2.0" effort="1000"/>
         </joint>
-        <joint name="${prefix}robotiq_85_right_knuckle_joint" type="revolute">
+        <joint name="${prefix}robotiq_85_right_knuckle_joint" type="continuous">
             <parent link="${prefix}robotiq_85_base_link"/>
             <child link="${prefix}robotiq_85_right_knuckle_link"/>
             <axis xyz="0 0 1"/>
             <origin rpy="0.0 0.0 0.0" xyz="0.05490451627 -0.03060114443 0.0"/>
-            <limit lower="-0.804" upper="0.0" velocity="2.0" effort="1000"/>
-            <mimic joint="${prefix}robotiq_85_left_knuckle_joint" multiplier="1"/>
-        </joint>
-        <gazebo>
-            <plugin name="${prefix}robotiq_85_right_knuckle_joint_mimic" filename="libroboticsgroup_gazebo_mimic_joint_plugin.so">
-                <joint>${prefix}robotiq_85_left_knuckle_joint</joint>
-                <mimicJoint>${prefix}robotiq_85_right_knuckle_joint</mimicJoint>
-            </plugin>
-            <plugin name="${prefix}robotiq_85_right_knuckle_link" filename="libroboticsgroup_gazebo_disable_link_plugin.so" >
-                <link>${prefix}robotiq_85_right_knuckle_link</link>
-            </plugin>
-        </gazebo>
+            <limit lower="-3.14" upper="3.14" velocity="100.0" effort="1000"/>
+            <mimic joint="${prefix}robotiq_85_left_knuckle_joint"/>
+        </joint>
         <link name="${prefix}robotiq_85_left_knuckle_link">
             <visual>
@@ -93,14 +84,10 @@
             <parent link="${prefix}robotiq_85_left_knuckle_link"/>
             <child link="${prefix}robotiq_85_left_finger_link"/>
-            <axis xyz="0 0 1"/>
             <origin xyz="-0.00408552455 -0.03148604435 0.0" rpy="0 0 0" />
-            <limit lower="0" upper="2.617994" velocity="2.0" effort="1000"/>
         </joint>
         <joint name="${prefix}robotiq_85_right_finger_joint" type="fixed">
             <parent link="${prefix}robotiq_85_right_knuckle_link"/>
             <child link="${prefix}robotiq_85_right_finger_link"/>
-            <axis xyz="0 0 1"/>
             <origin xyz="-0.00408552455 -0.03148604435 0.0" rpy="0 0 0" />
-            <limit lower="0" upper="2.617994" velocity="2.0" effort="0"/>
         </joint>
         <link name="${prefix}robotiq_85_left_finger_link">
@@ -142,38 +129,20 @@
             </inertial>
         </link>
-        <joint name="${prefix}robotiq_85_left_inner_knuckle_joint" type="revolute">
+        <joint name="${prefix}robotiq_85_left_inner_knuckle_joint" type="continuous">
             <parent link="${prefix}robotiq_85_base_link"/>
             <child link="${prefix}robotiq_85_left_inner_knuckle_link"/>
             <axis xyz="0 0 1"/>
             <origin xyz="0.06142 0.0127 0" rpy="${pi} 0.0 0.0" />
-            <limit lower="-0.804" upper="0.0" velocity="2.0" effort="1000"/>
+            <limit lower="-3.14" upper="3.14" velocity="100.0" effort="0.1"/>
             <mimic joint="${prefix}robotiq_85_left_knuckle_joint" offset="0"/>
         </joint>
-        <gazebo>
-            <plugin name="${prefix}robotiq_85_left_inner_knuckle_joint_mimic" filename="libroboticsgroup_gazebo_mimic_joint_plugin.so">
-                <joint>${prefix}robotiq_85_left_knuckle_joint</joint>
-                <mimicJoint>${prefix}robotiq_85_left_inner_knuckle_joint</mimicJoint>
-            </plugin>
-            <plugin name="${prefix}robotiq_85_left_inner_knuckle_link" filename="libroboticsgroup_gazebo_disable_link_plugin.so" >
-                <link>${prefix}robotiq_85_left_inner_knuckle_link</link>
-            </plugin>
-        </gazebo>
-        <joint name="${prefix}robotiq_85_right_inner_knuckle_joint" type="revolute">
+        <joint name="${prefix}robotiq_85_right_inner_knuckle_joint" type="continuous">
             <parent link="${prefix}robotiq_85_base_link"/>
             <child link="${prefix}robotiq_85_right_inner_knuckle_link"/>
             <axis xyz="0 0 1"/>
             <origin xyz="0.06142 -0.0127 0" rpy="0 0 0"/>
-            <limit lower="0" upper="0.804" velocity="2.0" effort="1000"/>
+            <limit lower="-3.14" upper="3.14" velocity="100.0" effort="0.1"/>
             <mimic joint="${prefix}robotiq_85_left_knuckle_joint" offset="0"/>
         </joint>
-        <gazebo>
-            <plugin name="${prefix}robotiq_85_right_inner_knuckle_joint_mimic" filename="libroboticsgroup_gazebo_mimic_joint_plugin.so">
-                <joint>${prefix}robotiq_85_left_knuckle_joint</joint>
-                <mimicJoint>${prefix}robotiq_85_right_inner_knuckle_joint</mimicJoint>
-            </plugin>
-            <plugin name="${prefix}robotiq_85_right_inner_knuckle_link" filename="libroboticsgroup_gazebo_disable_link_plugin.so" >
-                <link>${prefix}robotiq_85_right_inner_knuckle_link</link>
-            </plugin>
-        </gazebo>
         <link name="${prefix}robotiq_85_left_inner_knuckle_link">
             <visual>
@@ -214,40 +183,20 @@
             </inertial>
         </link>
-        <joint name="${prefix}robotiq_85_left_finger_tip_joint" type="revolute">
+        <joint name="${prefix}robotiq_85_left_finger_tip_joint" type="continuous">
             <parent link="${prefix}robotiq_85_left_inner_knuckle_link"/>
             <child link="${prefix}robotiq_85_left_finger_tip_link"/>
             <axis xyz="0 0 1"/>
             <origin xyz="0.04303959807 -0.03759940821 0.0" rpy="0.0 0.0 0.0"/>
-            <limit lower="0" upper="1.5707" velocity="2.0" effort="1000"/>
+            <limit lower="-3.14" upper="3.14" velocity="100.0" effort="0.1"/>
             <mimic joint="${prefix}robotiq_85_left_knuckle_joint" multiplier="-1"/>
         </joint>
-        <gazebo>
-            <plugin name="${prefix}${prefix}robotiq_85_left_finger_tip_joint_mimic" filename="libroboticsgroup_gazebo_mimic_joint_plugin.so">
-                <joint>${prefix}robotiq_85_left_knuckle_joint</joint>
-                <mimicJoint>${prefix}robotiq_85_left_finger_tip_joint</mimicJoint>
-                <multiplier>-1</multiplier>
-            </plugin>
-            <plugin name="${prefix}robotiq_85_left_finger_tip_link" filename="libroboticsgroup_gazebo_disable_link_plugin.so" >
-                <link>${prefix}robotiq_85_left_finger_tip_link</link>
-            </plugin>
-        </gazebo>
-        <joint name="${prefix}robotiq_85_right_finger_tip_joint" type="revolute">
+        <joint name="${prefix}robotiq_85_right_finger_tip_joint" type="continuous">
             <parent link="${prefix}robotiq_85_right_inner_knuckle_link"/>
             <child link="${prefix}robotiq_85_right_finger_tip_link"/>
             <axis xyz="0 0 1"/>
             <origin rpy="0.0 0.0 0.0" xyz="0.04303959807 -0.03759940821  0.0"/>
-            <limit lower="0" upper="1.5707" velocity="2.0" effort="1000"/>
+            <limit lower="-3.14" upper="3.14" velocity="100.0" effort="0.1"/>
             <mimic joint="${prefix}robotiq_85_left_knuckle_joint" multiplier="-1"/>
         </joint>
-        <gazebo>
-            <plugin name="${prefix}${prefix}robotiq_85_right_finger_tip_joint_mimic" filename="libroboticsgroup_gazebo_mimic_joint_plugin.so">
-                <joint>${prefix}robotiq_85_left_knuckle_joint</joint>
-                <mimicJoint>${prefix}robotiq_85_right_finger_tip_joint</mimicJoint>
-                <multiplier>-1</multiplier>
-            </plugin>
-            <plugin name="${prefix}robotiq_85_right_finger_tip_link" filename="libroboticsgroup_gazebo_disable_link_plugin.so" >
-                <link>${prefix}robotiq_85_right_finger_tip_link</link>
-            </plugin>
-        </gazebo>
         <link name="${prefix}robotiq_85_left_finger_tip_link">
             <visual>
