Commit message: major updates after integration
gazebo sim and moveit configuration also updated

File: vector_common/vector_description/urdf/sensors/kinect_one_sensor.urdf.xacro (robot description, xacro)
@@ -29,4 +29,11 @@
         </joint>
 	    <link name="${prefix}_link">
+            <inertial>
+                <mass value="0.1"/>
+                <origin xyz="0 0 0" rpy="0 0 0"/>
+                <inertia ixx="0.01"  ixy="0.0"  ixz="0.0"
+                         iyy="0.01"  iyz="0.0"
+                         izz="0.01" />
+            </inertial>
 			<visual>
 				<geometry>
@@ -40,64 +47,125 @@
 			</collision>
 		</link>
-        <link name="${prefix}_depth_frame"/>
-        <joint name="${prefix}_depth_joint" type="fixed">
+        <link name="${prefix}_ir_link">
+			<collision>
+				<geometry>
+					<sphere radius="0.0005"/>
+				</geometry>
+			</collision>
+            <inertial>
+                <mass value="0.1"/>
+                <origin xyz="0 0 0" rpy="0 0 0"/>
+                <inertia ixx="0.01"  ixy="0.0"  ixz="0.0"
+                         iyy="0.01"  iyz="0.0"
+                         izz="0.01" />
+            </inertial>
+        </link>
+        <joint name="${prefix}_ir_joint" type="fixed">
             <parent link="${prefix}_link"/>
-            <child link="${prefix}_depth_frame" />
-            <origin xyz="0 -0.02  0" rpy="0 0 0"/>
+            <child link="${prefix}_ir_link" />
+            <origin xyz="0.0245 -0.03325  0.04201" rpy="0 0 0"/>
         </joint>
-        <link name="${prefix}_rgb_frame"/>
+        <link name="${prefix}_ir_optical_frame"/>
+        <joint name="${prefix}_ir_optical_frame_joint" type="fixed">
+            <origin xyz="0 0 0" rpy="${-M_PI / 2.0} 0 ${-M_PI / 2.0}" />
+            <parent link="${prefix}_ir_link"/>
+            <child link="${prefix}_ir_optical_frame"/>
+        </joint>
+        <link name="${prefix}_rgb_link"/>
         <joint name="${prefix}_rgb_joint" type="fixed">
-            <parent link="${prefix}_link"/>
-            <child link="${prefix}_rgb_frame" />
-            <origin xyz="0 -0.045  0" rpy="0 0 0"/>
-        </joint>
-        <link name="${prefix}_depth_optical_frame"/>
-        <joint name="${prefix}_depth_optical_joint" type="fixed">
-            <parent link="${prefix}_depth_frame"/>
-            <child link="${prefix}_depth_optical_frame" />
-            <origin xyz="0 0 0" rpy="${-M_PI / 2.0} 0 ${-M_PI / 2.0}"/>
+            <parent link="${prefix}_ir_link"/>
+            <child link="${prefix}_rgb_link" />
+            <origin xyz="0 -0.06175  0" rpy="0 0 0"/>
         </joint>
         <link name="${prefix}_rgb_optical_frame"/>
         <joint name="${prefix}_rgb_optical_joint" type="fixed">
-            <parent link="${prefix}_rgb_frame"/>
+            <parent link="${prefix}_rgb_link"/>
             <child link="${prefix}_rgb_optical_frame" />
             <origin xyz="0 0 0" rpy="${-M_PI / 2.0} 0 ${-M_PI / 2.0}"/>
         </joint>
-        <gazebo reference="${prefix}_link">
-            <sensor type="depth" name="${prefix}">
+        <gazebo reference="${prefix}_ir_link">
+            <sensor type="depth" name="${prefix}_ir_sensor">
                 <always_on>true</always_on>
-                <update_rate>20.0</update_rate>
+                <update_rate>1.0</update_rate>
                 <camera>
-                    <horizontal_fov>${60.0*M_PI/180.0}</horizontal_fov>
+                    <horizontal_fov>${57.0*M_PI/180.0}</horizontal_fov>
                     <image>
-                        <format>R8G8B8</format>
+                        <format>L8</format>
                         <width>640</width>
                         <height>480</height>
                     </image>
                     <clip>
-                        <near>0.05</near>
-                        <far>8.0</far>
+                        <near>0.01</near>
+                        <far>5</far>
                     </clip>
                 </camera>
-                <plugin name="kinect_${prefix}_controller" filename="libgazebo_ros_openni_kinect.so">
-                    <cameraName>${prefix}</cameraName>
+                <plugin name="${prefix}_ir_link_controller" filename="libgazebo_ros_openni_kinect.so">
+                    <baseline>0.2</baseline>
                     <alwaysOn>true</alwaysOn>
-                    <updateRate>10</updateRate>
-                    <imageTopicName>rgb/image_raw</imageTopicName>
-                    <depthImageTopicName>depth/image_raw</depthImageTopicName>
-                    <pointCloudTopicName>depth/points</pointCloudTopicName>
-                    <cameraInfoTopicName>rgb/camera_info</cameraInfoTopicName>
-                    <depthImageCameraInfoTopicName>depth/camera_info</depthImageCameraInfoTopicName>
-                    <frameName>/vector/${prefix}_rgb_optical_frame</frameName>
-                    <baseline>0.1</baseline>
-                    <distortion_k1>0.0</distortion_k1>
-                    <distortion_k2>0.0</distortion_k2>
-                    <distortion_k3>0.0</distortion_k3>
-                    <distortion_t1>0.0</distortion_t1>
-                    <distortion_t2>0.0</distortion_t2>
-                    <pointCloudCutoff>0.4</pointCloudCutoff>
-                    <pointCloudCutoffMax>5.0</pointCloudCutoffMax>
+                    <updateRate>1.0</updateRate>
+                    <cameraName>${prefix}_ir</cameraName>
+                    <imageTopicName>/${prefix}/ir/image_raw</imageTopicName>
+                    <cameraInfoTopicName>/${prefix}/ir/camera_info</cameraInfoTopicName>
+                    <depthImageTopicName>/${prefix}/depth/image_raw</depthImageTopicName>
+                    <depthImageCameraInfoTopicName>/${prefix}/depth/camera_info</depthImageCameraInfoTopicName>
+                    <pointCloudTopicName>/${prefix}/depth/points</pointCloudTopicName>
+                    <frameName>${prefix}_ir_optical_frame</frameName>
+                    <pointCloudCutoff>0.5</pointCloudCutoff>
+                    <pointCloudCutoffMax>12.0</pointCloudCutoffMax>
+                    <distortionK1>0.0</distortionK1>
+                    <distortionK2>0.0</distortionK2>
+                    <distortionK3>0.0</distortionK3>
+                    <distortionT1>0.0</distortionT1>
+                    <distortionT2>0.0</distortionT2>
+                    <CxPrime>0</CxPrime>
+                    <Cx>0</Cx>
+                    <Cy>0</Cy>
+                    <focalLength>0</focalLength>
+                    <hackBaseline>0</hackBaseline>
                 </plugin>
             </sensor>
+            <material value="Gazebo/Red" />
+        </gazebo>
+        <gazebo reference="${prefix}_rgb_link">
+            <sensor type="depth" name="${prefix}_rgb_sensor">
+                <always_on>true</always_on>
+                <update_rate>1.0</update_rate>
+                <camera>
+                    <horizontal_fov>${57.0*M_PI/180.0}</horizontal_fov>
+                    <image>
+                        <format>B8G8R8</format>
+                        <width>640</width>
+                        <height>480</height>
+                    </image>
+                    <clip>
+                        <near>0.01</near>
+                        <far>5</far>
+                    </clip>
+                </camera>
+                <plugin name="${prefix}_rgb_link_controller" filename="libgazebo_ros_openni_kinect.so">
+                    <alwaysOn>true</alwaysOn>
+                    <updateRate>1.0</updateRate>
+                    <cameraName>${prefix}_rgb</cameraName>
+                    <imageTopicName>/${prefix}/rgb/image_raw</imageTopicName>
+                    <cameraInfoTopicName>/${prefix}/rgb/camera_info</cameraInfoTopicName>
+                    <depthImageTopicName>/${prefix}/depth/image_raw</depthImageTopicName>
+                    <depthImageCameraInfoTopicName>/${prefix}/depth/camera_info</depthImageCameraInfoTopicName>
+                    <pointCloudTopicName>/${prefix}/depth_registered/points</pointCloudTopicName>
+                    <frameName>${prefix}_rgb_optical_frame</frameName>
+                    <pointCloudCutoff>0.5</pointCloudCutoff>
+                    <pointCloudCutoffMax>12.0</pointCloudCutoffMax>
+                    <distortionK1>0.0</distortionK1>
+                    <distortionK2>0.0</distortionK2>
+                    <distortionK3>0.0</distortionK3>
+                    <distortionT1>0.0</distortionT1>
+                    <distortionT2>0.0</distortionT2>
+                    <CxPrime>0</CxPrime>
+                    <Cx>0</Cx>
+                    <Cy>0</Cy>
+                    <focalLength>0</focalLength>
+                    <hackBaseline>0</hackBaseline>
+                </plugin>
+            </sensor>
+            <material value="Gazebo/Red" />
         </gazebo>
     </xacro:macro>

File: vector_common/vector_description/urdf/sensors/pan_tilt_kinect_one.urdf.xacro (robot description, xacro)
@@ -41,20 +41,27 @@
 				</geometry>
 			</collision>
+            <inertial>
+                <mass value="0.1"/>
+                <origin xyz="0 0 0" rpy="0 0 0"/>
+                <inertia ixx="0.01"  ixy="0.0"  ixz="0.0"
+                         iyy="0.01"  iyz="0.0"
+                         izz="0.01" />
+            </inertial>
 		</link>
         <joint name="pan_joint" type="revolute">
             <origin xyz="0 0 0.0985" rpy="0 0 0" />
             <axis xyz="0 0 1"/>
-            <limit effort="6.0" lower="-1.570796326794897" upper="1.570796326794897" velocity="6.597"/>
             <parent link="pan_base_link" />
             <child link="pan_link" />
+            <limit effort="6.0" lower="-1.570796326794897" upper="1.570796326794897" velocity="6.597"/>
         </joint>
         <transmission name="pan_trans" type="SimpleTransmission">
 			<type>transmission_interface/SimpleTransmission</type>
+			<joint name="pan_joint">
+				<hardwareInterface>PositionJointInterface</hardwareInterface>
+			</joint>
 			<actuator name="pan_actuator">
 				<mechanicalReduction>1</mechanicalReduction>
 			</actuator>
-			<joint name="pan_joint">
-				<hardwareInterface>PositionJointInterface</hardwareInterface>
-			</joint>
 		</transmission>
 	    <link name="pan_link">
@@ -70,20 +77,27 @@
 				</geometry>
 			</collision>
+            <inertial>
+                <mass value="0.1"/>
+                <origin xyz="0 0 0" rpy="0 0 0"/>
+                <inertia ixx="0.01"  ixy="0.0"  ixz="0.0"
+                         iyy="0.01"  iyz="0.0"
+                         izz="0.01" />
+            </inertial>
 		</link>
         <joint name="tilt_joint" type="revolute">
             <origin xyz="0 0 0" rpy="0 0 0" />
             <axis xyz="0 1 0"/>
-            <limit effort="6.0" lower="-1.047197551196598" upper="1.570796326794897" velocity="6.597"/>
             <parent link="pan_link" />
             <child link="tilt_link" />
+            <limit effort="6.0" lower="-1.047197551196598" upper="1.570796326794897" velocity="6.597"/>
         </joint>
         <transmission name="tilt_trans" type="SimpleTransmission">
 			<type>transmission_interface/SimpleTransmission</type>
+			<joint name="tilt_joint">
+				<hardwareInterface>PositionJointInterface</hardwareInterface>
+			</joint>
 			<actuator name="tilt_actuator">
 				<mechanicalReduction>1</mechanicalReduction>
 			</actuator>
-			<joint name="tilt_joint">
-				<hardwareInterface>PositionJointInterface</hardwareInterface>
-			</joint>
 		</transmission>
 	    <link name="tilt_link">
@@ -98,4 +112,11 @@
 				</geometry>
 			</collision>
+            <inertial>
+                <mass value="0.1"/>
+                <origin xyz="0 0 0" rpy="0 0 0"/>
+                <inertia ixx="0.01"  ixy="0.0"  ixz="0.0"
+                         iyy="0.01"  iyz="0.0"
+                         izz="0.01" />
+            </inertial>
 		</link>
 		<xacro:kinect_one_sensor prefix="${rgbd_prefix}" parent="tilt_link">

File: vector_common/vector_description/urdf/vector.urdf.xacro (robot description, xacro)
@@ -46,10 +46,25 @@
         <origin xyz="0.22806971 0 0.46024800" rpy="0 0 0" />
     </xacro:vector_linear_actuator>
-    <xacro:jaco_robot prefix="jaco_" parent="linear_actuator_link">
-        <origin xyz="0.06079866 0 0" rpy="${M_PI/2} 0 ${M_PI/2}"/>
-    </xacro:jaco_robot>
-    <xacro:robotiq_85_gripper prefix="jaco_" parent="jaco_ee_link" >
-        <origin xyz="0 0 0" rpy="0 0 0"/>
-    </xacro:robotiq_85_gripper>
+    <!-- Arms -->
+    <xacro:if value="$(optenv VECTOR_HAS_KINOVA_ARM false)">
+        <xacro:jaco_robot prefix="right_" parent="linear_actuator_link">
+            <origin xyz="0.06079866 0 0" rpy="${M_PI/2} 0 ${M_PI/2}"/>
+        </xacro:jaco_robot>
+        <xacro:if value="$(optenv VECTOR_HAS_TWO_KINOVA_ARMS false)">
+            <xacro:jaco_robot prefix="left_" parent="linear_actuator_link">
+                <origin xyz="0.06079866 0 0" rpy="${M_PI/2} 0 ${M_PI/2}"/>
+            </xacro:jaco_robot>
+        </xacro:if>
+        <xacro:if value="$(optenv VECTOR_HAS_ROBOTIQ_GRIPPER false)">
+            <xacro:robotiq_85_gripper prefix="right_" parent="right_ee_link" >
+                <origin xyz="0 0 0" rpy="0 0 0"/>
+            </xacro:robotiq_85_gripper>
+            <xacro:if value="$(optenv VECTOR_HAS_TWO_ROBOTIQ_GRIPPERS false)">
+                <xacro:robotiq_85_gripper prefix="left_" parent="right_ee_link" >
+                    <origin xyz="0 0 0" rpy="0 0 0"/>
+                </xacro:robotiq_85_gripper>
+            </xacro:if>
+        </xacro:if>
+    </xacro:if>
     <!-- Setup any accessories defined in the environment -->
     <xacro:vector_accessories />

Commit message: updated noise and drift characterists for simulation

File: vector_common/vector_description/urdf/accessories.urdf.xacro (robot description, xacro)
@@ -40,10 +40,10 @@
                 <bodyName>sic_imu_frame</bodyName>
                 <topicName>/vector/feedback/sic_imu</topicName>
-                <accelDrift>0.005 0.005 0.005</accelDrift>
-                <accelGaussianNoise>0.005 0.005 0.005</accelGaussianNoise>
-                <rateDrift>0.005 0.005 0.005 </rateDrift>
-                <rateGaussianNoise>0.005 0.005 0.005 </rateGaussianNoise>
-                <headingDrift>0.005</headingDrift>
-                <headingGaussianNoise>0.005</headingGaussianNoise>
+                <accelDrift>0.0005 0.0005 0.0005</accelDrift>
+                <accelGaussianNoise>0.0005 0.0005 0.0005</accelGaussianNoise>
+                <rateDrift>0.0005 0.0005 0.0005</rateDrift>
+                <rateGaussianNoise>0.00005 0.00005 0.00005 </rateGaussianNoise>
+                <headingDrift>0.00005</headingDrift>
+                <headingGaussianNoise>0.00005</headingGaussianNoise>
             </plugin>
         </gazebo>
@@ -62,10 +62,10 @@
                     <bodyName>ext_imu_frame</bodyName>
                     <topicName>/vector/feedback/ext_imu</topicName>
-                    <accelDrift>0.005 0.005 0.005</accelDrift>
-                    <accelGaussianNoise>0.005 0.005 0.005</accelGaussianNoise>
-                    <rateDrift>0.005 0.005 0.005 </rateDrift>
-                    <rateGaussianNoise>0.005 0.005 0.005 </rateGaussianNoise>
-                    <headingDrift>0.005</headingDrift>
-                    <headingGaussianNoise>0.005</headingGaussianNoise>
+	                <accelDrift>0.0005 0.0005 0.0005</accelDrift>
+	                <accelGaussianNoise>0.0005 0.0005 0.0005</accelGaussianNoise>
+	                <rateDrift>0.0005 0.0005 0.0005</rateDrift>
+	                <rateGaussianNoise>0.00005 0.00005 0.00005 </rateGaussianNoise>
+	                <headingDrift>0.00005</headingDrift>
+	                <headingGaussianNoise>0.00005</headingGaussianNoise>
                 </plugin>
             </gazebo>
@@ -85,6 +85,9 @@
         <!-- Hokuyo UST-20LX Sensor -->
         <xacro:if value="$(optenv VECTOR_HAS_HOKUYO false)">
-            <xacro:hokuyo_ust20lx laser_prefix="base" parent="$(optenv VECTOR_PARENT_LINK base_chassis_link)">
-                <origin xyz="$(optenv HOKUYO_XYZ 0.35 0 0.2)" rpy="$(optenv HOKUYO_RPY 3.14159 0 0)" />
+            <xacro:hokuyo_ust20lx laser_prefix="front" parent="$(optenv VECTOR_PARENT_LINK base_chassis_link)">
+                <origin xyz="$(optenv HOKUYO_FRONT_XYZ 0.35 0 0.2)" rpy="$(optenv HOKUYO_FRONT_RPY 3.14159 0 0)" />
+            </xacro:hokuyo_ust20lx>
+            <xacro:hokuyo_ust20lx laser_prefix="rear" parent="$(optenv VECTOR_PARENT_LINK base_chassis_link)">
+                <origin xyz="$(optenv HOKUYO_REAR_XYZ -0.35 0 0.2)" rpy="$(optenv HOKUYO_REAR_RPY 3.14159 0 3.14159)" />
             </xacro:hokuyo_ust20lx>
         </xacro:if>

Commit message: removed second laser for a different project, will formally add support for multilaser at some point

File: vector_common/vector_description/urdf/accessories.urdf.xacro (robot description, xacro)
@@ -85,9 +85,6 @@
         <!-- Hokuyo UST-20LX Sensor -->
         <xacro:if value="$(optenv VECTOR_HAS_HOKUYO false)">
-            <xacro:hokuyo_ust20lx laser_prefix="front" parent="$(optenv VECTOR_PARENT_LINK base_chassis_link)">
-                <origin xyz="$(optenv HOKUYO_FRONT_XYZ 0.35 0 0.2)" rpy="$(optenv HOKUYO_FRONT_RPY 3.14159 0 0)" />
-            </xacro:hokuyo_ust20lx>
-            <xacro:hokuyo_ust20lx laser_prefix="rear" parent="$(optenv VECTOR_PARENT_LINK base_chassis_link)">
-                <origin xyz="$(optenv HOKUYO_REAR_XYZ -0.35 0 0.2)" rpy="$(optenv HOKUYO_REAR_RPY 3.14159 0 3.14159)" />
+            <xacro:hokuyo_ust20lx laser_prefix="base" parent="$(optenv VECTOR_PARENT_LINK base_chassis_link)">
+                <origin xyz="$(optenv HOKUYO_XYZ 0.35 0 0.2)" rpy="$(optenv HOKUYO_RPY 3.14159 0 0)" />
             </xacro:hokuyo_ust20lx>
         </xacro:if>

Commit message: making updates to the navigation demos so they are setup for vector.
Removed 3D for now until I have time to set it up. It was not using the most current 3D packages and is more effort to update

Added playpen example for sim

Updated vector_viz configurations

Updated laser naming to prepare for multiple laser support

Fixed issue with interactive marker and simulation not having a timeout when the user stops interacting with the teleop marker. Robot now stops after a 0.4 sec timeout.

File: vector_common/vector_description/urdf/accessories.urdf.xacro (robot description, xacro)
@@ -79,7 +79,7 @@
         <!-- SICK LMS1XX Sensor -->
         <xacro:if value="$(optenv VECTOR_HAS_SICK_TIM false)">
-            <xacro:sick_lms1xx laser_prefix="base" parent="$(optenv VECTOR_PARENT_LINK base_chassis_link)">
+            <xacro:hokuyo_ust20lx laser_prefix="base" parent="$(optenv VECTOR_PARENT_LINK base_chassis_link)">
                 <origin xyz="$(optenv SICK_TIM_XYZ 0 0 1.0)" rpy="$(optenv SICK_TIM_RPY 3.14159 0 0)" />
-            </xacro:sick_lms1xx>
+            </xacro:hokuyo_ust20lx>
         </xacro:if>
         <!-- Hokuyo UST-20LX Sensor -->

File: vector_common/vector_description/urdf/sensors/hokuyo_ust20lx.urdf.xacro (robot description, xacro)
@@ -41,5 +41,5 @@
         </link>
         <gazebo reference="${laser_prefix}_laser_link">
-            <sensor type="ray" name="${laser_prefix}_hokuyo_laser">
+            <sensor type="ray" name="${laser_prefix}_laser">
                 <pose>0 0 0 0 0 0</pose>
                 <visualize>false</visualize>
@@ -65,6 +65,6 @@
                     </noise>
                 </ray>
-                <plugin name="hokuyo_node" filename="libgazebo_ros_laser.so">
-                    <topicName>/vector/${laser_prefix}_scan</topicName>
+                <plugin name="gazebo_laser_node" filename="libgazebo_ros_laser.so">
+                    <topicName>/vector/${laser_prefix}_scan_filtered</topicName>
                     <frameName>${laser_prefix}_laser_link</frameName>
                 </plugin>

File: vector_common/vector_description/urdf/vector.urdf.xacro (robot description, xacro)
@@ -33,17 +33,23 @@
           <robotNamespace>/</robotNamespace>
         </plugin>
-        <plugin name="object_controller" filename="libgazebo_ros_planar_move.so">
+        <plugin name="object_controller" filename="libgazebo_ros_force_based_move.so">
             <commandTopic>/vector/cmd_vel</commandTopic>
             <odometryTopic>/vector/feedback/wheel_odometry</odometryTopic>
             <odometryFrame>odom</odometryFrame>
-            <odometryRate>100</odometryRate>
+            <odometryRate>30.0</odometryRate>
             <robotBaseFrame>base_link</robotBaseFrame>
+            <publishOdometryTf>0</publishOdometryTf>
+            <yaw_velocity_p_gain>10000.0</yaw_velocity_p_gain>
+            <x_velocity_p_gain>10000.0</x_velocity_p_gain>
+            <y_velocity_p_gain>10000.0</y_velocity_p_gain>
         </plugin>
     </gazebo>
     <xacro:vector_base name="base"/>
     <!--linear actuator-->
-    <xacro:vector_linear_actuator parent="base_chassis_link">
-        <origin xyz="0.22806971 0 0.46024800" rpy="0 0 0" />
-    </xacro:vector_linear_actuator>
+    <xacro:if value="$(optenv VECTOR_HAS_LINEAR_ACTUATOR false)">
+        <xacro:vector_linear_actuator parent="base_chassis_link">
+            <origin xyz="0.22806971 0 0.46024800" rpy="0 0 0" />
+        </xacro:vector_linear_actuator>
+    </xacro:if>
     <!-- Arms -->
     <xacro:if value="$(optenv VECTOR_HAS_KINOVA_ARM false)">

File: vector_common/vector_description/urdf/vector_components/vector_base.urdf.xacro (robot description, xacro)
@@ -27,4 +27,7 @@
         <!-- Base link is the center of the robot's chassis between the motors projected on the ground -->
         <link name="${name}_link"/>
+        <gazebo reference="base_link">
+            <mu1>0.0</mu1>
+        </gazebo>
         <joint name="${name}_chassis_joint" type="fixed">
             <origin xyz="0 0 ${wheel_radius}" rpy="0 0 0" />
@@ -52,4 +55,7 @@
 			</visual>
 		</link>
+        <gazebo reference="base_chassis_link">
+            <mu1>0.0</mu1>
+        </gazebo>
     </xacro:macro>
 </robot>

Commit message: forgot one file from prev checkin:
updating to include exoskeleton and fix collision model for final skins

File: vector_common/vector_description/urdf/accessories.urdf.xacro (robot description, xacro)
@@ -74,5 +74,5 @@
         <xacro:if value="$(optenv VECTOR_HAS_KINECT_PAN_TILT false)">
             <xacro:pan_tilt_kinect_one rgbd_prefix="kinect" parent="$(optenv KINECT_PAN_TILT_PARENT_LINK base_chassis_link)">
-                <origin xyz="$(optenv KINECT_PAN_TILT_XYZ 0.16688476 0 0.96899800)" rpy="$(optenv KINECT_PAN_TILT_RPY 0 0 0)" />
+                <origin xyz="$(optenv KINECT_PAN_TILT_XYZ 0.16688476 0 0.99465201)" rpy="$(optenv KINECT_PAN_TILT_RPY 0 0 0)" />
             </xacro:pan_tilt_kinect_one>
         </xacro:if>
