Commit message: Please review vector_config.sh and make sure it matches your machine setup. THere have been a few changes to accomodate multi-laser support
updating the master to fix the force based move plugin odometry and continue support for robot_localization in sim

the environment variable in vector_config.sh VECTOR_USE_PLATFORM_ODOMETRY controls simulation odometry. If true the sim will use gazebo ground truth, if false robot_localization with ground truth fused.

Added support for 2 lasers in vector_config.sh. You will need to update it to match the configuration of the machine

added separate jaco only sim launch files and moveit test

added sick_tim support now that it is standard (you will need to run 'sudo apt-get install ros-indigo-sick-tim)

File: vector_common/vector_description/urdf/accessories.urdf.xacro (robot description, xacro)
@@ -22,5 +22,5 @@
 -->
 <robot name="vector_accessories" xmlns:xacro="http://ros.org/wiki/xacro">
-    <xacro:include filename="$(find vector_description)/urdf/sensors/sick_lms1xx.urdf.xacro"/>
+    <xacro:include filename="$(find vector_description)/urdf/sensors/sick_tim.urdf.xacro"/>
     <xacro:include filename="$(find vector_description)/urdf/sensors/hokuyo_ust20lx.urdf.xacro"/>
     <xacro:include filename="$(find vector_description)/urdf/sensors/pgr_flea3.urdf.xacro"/>
@@ -77,15 +77,31 @@
             </xacro:pan_tilt_kinect_one>
         </xacro:if>
-        <!-- SICK LMS1XX Sensor -->
-        <xacro:if value="$(optenv VECTOR_HAS_SICK_TIM false)">
-            <xacro:hokuyo_ust20lx laser_prefix="base" parent="$(optenv VECTOR_PARENT_LINK base_chassis_link)">
-                <origin xyz="$(optenv SICK_TIM_XYZ 0 0 1.0)" rpy="$(optenv SICK_TIM_RPY 3.14159 0 0)" />
-            </xacro:hokuyo_ust20lx>
+        <!-- First laser Sensor -->
+        <xacro:if value="$(optenv VECTOR_HAS_ONE_2D_LASER false)">
+            <!-- SICK TIM Sensor -->
+            <xacro:if value="$(optenv VECTOR_LASER1_IS_SICK_TIM false)">
+                <xacro:sick_tim laser_prefix="$(optenv LASER1_PREFIX base)" parent="$(optenv VECTOR_PARENT_LINK base_chassis_link)">
+                    <origin xyz="$(optenv LASER1_XYZ 0.35 0 0.2)" rpy="$(optenv LASER1_RPY 3.14159 0 0)" />
+                </xacro:sick_tim>
+            </xacro:if>
+            <xacro:if value="$(optenv VECTOR_LASER1_IS_HOKUYO false)">
+                <xacro:hokuyo_ust20lx laser_prefix="$(optenv LASER1_PREFIX base)" parent="$(optenv VECTOR_PARENT_LINK base_chassis_link)">
+                    <origin xyz="$(optenv LASER1_XYZ 0.35 0 0.2)" rpy="$(optenv LASER1_RPY 3.14159 0 0)" />
+                </xacro:hokuyo_ust20lx>
+            </xacro:if>
         </xacro:if>
-        <!-- Hokuyo UST-20LX Sensor -->
-        <xacro:if value="$(optenv VECTOR_HAS_HOKUYO false)">
-            <xacro:hokuyo_ust20lx laser_prefix="base" parent="$(optenv VECTOR_PARENT_LINK base_chassis_link)">
-                <origin xyz="$(optenv HOKUYO_XYZ 0.35 0 0.2)" rpy="$(optenv HOKUYO_RPY 3.14159 0 0)" />
-            </xacro:hokuyo_ust20lx>
+        <!-- Second laser Sensor -->
+        <xacro:if value="$(optenv VECTOR_HAS_SECOND_2D_LASER false)">
+            <!-- SICK TIM Sensor -->
+            <xacro:if value="$(optenv VECTOR_LASER2_IS_SICK_TIM false)">
+                <xacro:sick_tim laser_prefix="$(optenv LASER2_PREFIX base)" parent="$(optenv VECTOR_PARENT_LINK base_chassis_link)">
+                    <origin xyz="$(optenv LASER2_XYZ 0.35 0 0.2)" rpy="$(optenv LASER2_RPY 3.14159 0 0)" />
+                </xacro:sick_tim>
+            </xacro:if>
+            <xacro:if value="$(optenv VECTOR_LASER2_IS_HOKUYO false)">
+                <xacro:hokuyo_ust20lx laser_prefix="$(optenv LASER2_PREFIX base)" parent="$(optenv VECTOR_PARENT_LINK base_chassis_link)">
+                    <origin xyz="$(optenv LASER2_XYZ 0.35 0 0.2)" rpy="$(optenv LASER2_RPY 3.14159 0 0)" />
+                </xacro:hokuyo_ust20lx>
+            </xacro:if>
         </xacro:if>
         <!-- PGR FLEA3 Sensor -->

File: vector_common/vector_description/urdf/vector.urdf.xacro (robot description, xacro)
@@ -29,20 +29,40 @@
     <xacro:include filename="$(find vector_description)/urdf/manipulation/robotiq/robotiq_85_gripper.urdf.xacro" />
     <xacro:property name="M_PI" value="3.14159"/>
-    <gazebo>
-        <plugin name="gazebo_ros_control" filename="libgazebo_ros_control.so">
-          <robotNamespace>/</robotNamespace>
-        </plugin>
-        <plugin name="object_controller" filename="libgazebo_ros_force_based_move.so">
-            <commandTopic>/vector/cmd_vel</commandTopic>
-            <odometryTopic>/vector/feedback/wheel_odometry</odometryTopic>
-            <odometryFrame>odom</odometryFrame>
-            <odometryRate>30.0</odometryRate>
-            <robotBaseFrame>base_link</robotBaseFrame>
-            <publishOdometryTf>0</publishOdometryTf>
-            <yaw_velocity_p_gain>100.0</yaw_velocity_p_gain>
-            <x_velocity_p_gain>10000.0</x_velocity_p_gain>
-            <y_velocity_p_gain>10000.0</y_velocity_p_gain>
-        </plugin>
-    </gazebo>
+    <xacro:if value="$(optenv VECTOR_USE_PLATFORM_ODOMETRY false)">
+        <gazebo>
+            <plugin name="gazebo_ros_control" filename="libgazebo_ros_control.so">
+              <robotNamespace>/</robotNamespace>
+            </plugin>
+            <plugin name="object_controller" filename="libgazebo_ros_force_based_move.so">
+                <commandTopic>/vector/cmd_vel</commandTopic>
+                <odometryTopic>/vector/odometry/local_filtered</odometryTopic>
+                <odometryFrame>odom</odometryFrame>
+                <odometryRate>30.0</odometryRate>
+                <robotBaseFrame>base_link</robotBaseFrame>
+                <publishOdometryTf>1</publishOdometryTf>
+                <yaw_velocity_p_gain>100.0</yaw_velocity_p_gain>
+                <x_velocity_p_gain>10000.0</x_velocity_p_gain>
+                <y_velocity_p_gain>10000.0</y_velocity_p_gain>
+            </plugin>
+        </gazebo>
+    </xacro:if>
+    <xacro:unless value="$(optenv VECTOR_USE_PLATFORM_ODOMETRY false)">
+        <gazebo>
+            <plugin name="gazebo_ros_control" filename="libgazebo_ros_control.so">
+              <robotNamespace>/</robotNamespace>
+            </plugin>
+            <plugin name="object_controller" filename="libgazebo_ros_force_based_move.so">
+                <commandTopic>/vector/cmd_vel</commandTopic>
+                <odometryTopic>/vector/feedback/wheel_odometry</odometryTopic>
+                <odometryFrame>odom</odometryFrame>
+                <odometryRate>30.0</odometryRate>
+                <robotBaseFrame>base_link</robotBaseFrame>
+                <publishOdometryTf>0</publishOdometryTf>
+                <yaw_velocity_p_gain>100.0</yaw_velocity_p_gain>
+                <x_velocity_p_gain>10000.0</x_velocity_p_gain>
+                <y_velocity_p_gain>10000.0</y_velocity_p_gain>
+            </plugin>
+        </gazebo>
+    </xacro:unless>
     <xacro:vector_base name="base"/>
     <!--linear actuator-->
