Commit message: updated arm origin

File: vector_common/vector_description/urdf/vector_7dof.urdf.xacro (robot description, xacro)
@@ -74,14 +74,8 @@
     <!-- Arms -->
     <xacro:if value="$(optenv VECTOR_HAS_KINOVA_ARM false)">
-        <xacro:j2s7s300 base_parent="linear_actuator_link">
-            <xacro:if value="$(optenv VECTOR_HAS_TWO_KINOVA_ARMS false)">
-                <origin xyz="0.06079866 -0.1319 0" rpy="${M_PI/2} ${M_PI/2} ${M_PI/2}"/>
-            </xacro:if>
-        </xacro:j2s7s300>
-        <xacro:if value="$(optenv VECTOR_HAS_TWO_KINOVA_ARMS false)">
-            <xacro:j2s7s300 base_parent="linear_actuator_link">
-                <origin xyz="0.06079866 0.1319 0" rpy="${M_PI/2} 0 ${M_PI/2}"/>
-            </xacro:j2s7s300>
-        </xacro:if>
+        <xacro:j2s7s300 base_parent="linear_actuator_link" >
+	    <!-- Note: origin is overwritten in kinova urdf -->
+            <origin xyz="0 0 0" rpy="0 0 0" />
+	</xacro:j2s7s300>
     </xacro:if>
     <!-- Setup any accessories defined in the environment -->

Commit message: Initial commit

File: vector_common/vector_description/urdf/vector_7dof.urdf.xacro (robot description, xacro)
@@ -26,5 +26,6 @@
     <xacro:include filename="$(find vector_description)/urdf/linear_actuator/vector_linear_actuator.urdf.xacro" />
     <xacro:include filename="$(find vector_description)/urdf/accessories.urdf.xacro" />
-    <xacro:include filename="$(find kinova_description)/urdf/j2s7s300.xacro" />
+    <xacro:include filename="$(find kinova_description)/urdf/j2s7s300_mod.xacro" />
+    <xacro:include filename="$(find vector_description)/urdf/manipulation/robotiq/robotiq_85_gripper.urdf.xacro" />
     <xacro:property name="M_PI" value="3.14159"/>
     <xacro:if value="$(optenv VECTOR_USE_PLATFORM_ODOMETRY false)">
@@ -73,9 +74,35 @@
     </xacro:if>
     <!-- Arms -->
+    <!-- <xacro:if value="$(optenv VECTOR_HAS_KINOVA_ARM false)">
+        <xacro:j2s7s300 base_parent="linear_actuator_link" > -->
+	    <!-- Note: origin is overwritten in kinova urdf -->
+           <!-- <origin xyz="0 0 0" rpy="0 0 0" />
+	</xacro:j2s7s300>
+    </xacro:if> -->
     <xacro:if value="$(optenv VECTOR_HAS_KINOVA_ARM false)">
-        <xacro:j2s7s300 base_parent="linear_actuator_link" >
-	    <!-- Note: origin is overwritten in kinova urdf -->
-            <origin xyz="0 0 0" rpy="0 0 0" />
-	</xacro:j2s7s300>
+	<xacro:j2s7s300 prefix="right" base_parent="linear_actuator_link" origin_xyz="0.06079866 -0.1319 0" origin_rpy="${M_PI/2} 0 ${M_PI/2}" />
+        <!--<xacro:j2s7s300 prefix="right_" base_parent="linear_actuator_link">
+            <xacro:unless value="$(optenv VECTOR_HAS_TWO_KINOVA_ARMS false)">
+		<xacro:property name="origin_xyz" value="0.06079866 0 0" />
+		<xacro:property name="origin_rpy" value="${M_PI/2} 0 ${M_PI/2}" />
+            </xacro:unless>
+            <xacro:if value="$(optenv VECTOR_HAS_TWO_KINOVA_ARMS false)">
+		<xacro:property name="origin_xyz" value="0.06079866 -0.1319 0" />
+		<xacro:property name="origin_rpy" value="${M_PI/2} 0 ${M_PI/2}" />
+            </xacro:if>
+        </xacro:j2s7s300>-->
+        <xacro:if value="$(optenv VECTOR_HAS_TWO_KINOVA_ARMS false)">
+            <xacro:j2s7s300 prefix="left" base_parent="linear_actuator_link" origin_xyz="0.06079866 0.1319 0" origin_rpy="${M_PI/2} 0 ${M_PI/2}" />
+        </xacro:if>
+        <xacro:if value="$(optenv VECTOR_HAS_ROBOTIQ_GRIPPER false)">
+            <xacro:robotiq_85_gripper prefix="right_" parent="right_link_6" >
+                <origin xyz="0 0.10375 0" rpy="-${M_PI/2} 0 ${M_PI/2}"/>
+            </xacro:robotiq_85_gripper>
+            <xacro:if value="$(optenv VECTOR_HAS_TWO_ROBOTIQ_GRIPPERS false)">
+                <xacro:robotiq_85_gripper prefix="left_" parent="left_link_6" >
+                    <origin xyz="0 0.10375 0" rpy="-${M_PI/2} 0 ${M_PI/2}"/>
+                </xacro:robotiq_85_gripper>
+            </xacro:if>
+        </xacro:if>
     </xacro:if>
     <!-- Setup any accessories defined in the environment -->

Commit message: Minor updates in urdf

File: vector_common/vector_description/urdf/vector_7dof.urdf.xacro (robot description, xacro)
@@ -26,5 +26,5 @@
     <xacro:include filename="$(find vector_description)/urdf/linear_actuator/vector_linear_actuator.urdf.xacro" />
     <xacro:include filename="$(find vector_description)/urdf/accessories.urdf.xacro" />
-    <xacro:include filename="$(find vector_description)/urdf/manipulation/jaco/j2s7s300_mod.xacro" />
+    <xacro:include filename="$(find vector_description)/urdf/manipulation/jaco/j2s7s300.xacro" />
     <xacro:include filename="$(find vector_description)/urdf/manipulation/robotiq/robotiq_85_gripper.urdf.xacro" />
     <xacro:property name="M_PI" value="3.14159"/>
@@ -74,25 +74,22 @@
     </xacro:if>
     <!-- Arms -->
-    <!-- <xacro:if value="$(optenv VECTOR_HAS_KINOVA_ARM false)">
-        <xacro:j2s7s300 base_parent="linear_actuator_link" > -->
-	    <!-- Note: origin is overwritten in kinova urdf -->
-           <!-- <origin xyz="0 0 0" rpy="0 0 0" />
-	</xacro:j2s7s300>
-    </xacro:if> -->
-    <xacro:if value="$(optenv VECTOR_HAS_KINOVA_ARM false)">
-		<xacro:j2s7s300 prefix="right" base_parent="linear_actuator_link" origin_xyz="0.06079866 -0.1319 0" origin_rpy="${M_PI/2} 0 ${M_PI/2}" />
-        <!--<xacro:j2s7s300 prefix="right_" base_parent="linear_actuator_link">
-            <xacro:unless value="$(optenv VECTOR_HAS_TWO_KINOVA_ARMS false)">
-		<xacro:property name="origin_xyz" value="0.06079866 0 0" />
-		<xacro:property name="origin_rpy" value="${M_PI/2} 0 ${M_PI/2}" />
-            </xacro:unless>
-            <xacro:if value="$(optenv VECTOR_HAS_TWO_KINOVA_ARMS false)">
-		<xacro:property name="origin_xyz" value="0.06079866 -0.1319 0" />
-		<xacro:property name="origin_rpy" value="${M_PI/2} 0 ${M_PI/2}" />
-            </xacro:if>
-        </xacro:j2s7s300>-->
-        <xacro:if value="$(optenv VECTOR_HAS_TWO_KINOVA_ARMS false)">
+	<xacro:unless value="$(optenv VECTOR_HAS_TWO_KINOVA_ARMS false)">
+		<xacro:if value="$(optenv VECTOR_HAS_KINOVA_ARM false)">
+		    <xacro:j2s7s300 base_parent="linear_actuator_link" >
+			<!-- Note: origin is overwritten in kinova urdf -->
+		       <origin xyz="0 0 0" rpy="0 0 0" />
+			</xacro:j2s7s300>
+		</xacro:if>
+		<xacro:if value="$(optenv VECTOR_HAS_ROBOTIQ_GRIPPER false)">
+            <xacro:robotiq_85_gripper prefix="right_" parent="right_link_7" >
+                <!-- <origin xyz="0 0.10375 0" rpy="-${M_PI/2} 0 ${M_PI/2}"/> -->
+				<origin xyz="0 0 0" rpy="0 ${M_PI/2} 0"/>
+            </xacro:robotiq_85_gripper>
+		</xacro:if>
+	</xacro:unless>
+	<!-- Two Arms -->
+	<xacro:if value="$(optenv VECTOR_HAS_TWO_KINOVA_ARMS false)">
+			<xacro:j2s7s300 prefix="right" base_parent="linear_actuator_link" origin_xyz="0.06079866 -0.1319 0" origin_rpy="${M_PI/2} 0 ${M_PI/2}" />
             <xacro:j2s7s300 prefix="left" base_parent="linear_actuator_link" origin_xyz="0.06079866 0.1319 0" origin_rpy="${M_PI/2} 0 ${M_PI/2}" />
-        </xacro:if>
         <xacro:if value="$(optenv VECTOR_HAS_ROBOTIQ_GRIPPER false)">
             <xacro:robotiq_85_gripper prefix="right_" parent="right_link_7" >

Commit message: change so that we load the kinova arm in a consistent method with nimbus

File: vector_common/vector_description/urdf/vector_7dof.urdf.xacro (robot description, xacro)
@@ -74,7 +74,7 @@
     <!-- Arms -->
     <xacro:if value="$(optenv VECTOR_HAS_KINOVA_ARM false)">
-        <xacro:j2s7s300 base_parent="linear_actuator_link" >
+        <xacro:j2s7s300 base_parent="linear_actuator_link" trans="0.06079866 0 0" rot="${J_PI/2} 0 ${J_PI/2}">
 	    <!-- Note: origin is overwritten in kinova urdf -->
-            <origin xyz="0 0 0" rpy="0 0 0" />
+            <origin xyz="0.06079866 0 0" rpy="${J_PI/2} 0 ${J_PI/2}" />
 	</xacro:j2s7s300>
     </xacro:if>
