Commit message: updating to include exoskeleton and fix collision model for final skins

File: vector_common/vector_description/urdf/sensors/pan_tilt_kinect_one.urdf.xacro (robot description, xacro)
@@ -72,5 +72,5 @@
 			</visual>
 			<collision>
-			    <origin xyz="0 0 -0.0985" rpy="0 0 0" />
+			    <origin xyz="0 0 0" rpy="0 0 0" />
 				<geometry>
 					<mesh filename="package://vector_description/meshes/sensors/collision/tilt_actuator_collision.STL" />

Commit message: Set offset to correct for pan joint angle

File: vector_common/vector_description/urdf/sensors/pan_tilt_kinect_one.urdf.xacro (robot description, xacro)
@@ -50,5 +50,6 @@
 		</link>
         <joint name="pan_joint" type="revolute">
-            <origin xyz="0 0 0.0985" rpy="0 0 0" />
+            <!-- <origin xyz="0 0 0.0985" rpy="0 0 0" /> -->
+            <origin xyz="0 0 0.0985" rpy="0 0 0.772" />
             <axis xyz="0 0 1"/>
             <parent link="pan_base_link" />

Commit message: corercted pan tilt tf tree

File: vector_common/vector_description/urdf/sensors/pan_tilt_kinect_one.urdf.xacro (robot description, xacro)
@@ -50,5 +50,5 @@
 		</link>
         <joint name="pan_joint" type="revolute">
-            <origin xyz="0 0 0.0985" rpy="0 0 0" />
+            <origin xyz="0 0 0.0985" rpy="0 0 0.787" />
             <axis xyz="0 0 1"/>
             <parent link="pan_base_link" />
