Commit message: updated urdf

File: vector_common/vector_description/urdf/manipulation/jaco/j2s7s300_mod.xacro (robot description, xacro)
@@ -87,5 +87,4 @@
     <property name="joint_6_lower_limit" value="${30/180*J_PI}" />
     <property name="joint_6_upper_limit" value="${330/180*J_PI}" />
-	<!--
     <property name="joint_7" value="joint_7" />
     <property name="joint_7_type" value="continuous" />
@@ -95,4 +94,5 @@
     <property name="joint_7_lower_limit" value="${-2*J_PI}" />
     <property name="joint_7_upper_limit" value="${2*J_PI}" />
+	<!--
     <property name="joint_end_effector" value="end_effector_offset" />
     <property name="joint_end_effector_type" value="fixed" />
@@ -100,8 +100,10 @@
     <property name="joint_end_effector_origin_xyz" value="0 0 -0.1600" />
     <property name="joint_end_effector_origin_rpy" value="${J_PI} 0 0" /> -->
-    <xacro:macro name="j2s7s300" params="base_parent prefix:=j2s7s300">
-        <xacro:gazebo_config robot_namespace="${prefix}"/>
+    <xacro:macro name="j2s7s300" params="base_parent prefix origin_xyz origin_rpy">
+        <!--xacro:gazebo_config robot_namespace="${prefix}"/> -->
+        <xacro:gazebo_config robot_namespace="/"/>
         <xacro:kinova_armlink link_name="${prefix}_link_base" link_mesh="${link_base_mesh}" mesh_no="${link_base_mesh_no}"/>
-        <xacro:kinova_armjoint joint_name="${prefix}_joint_base" type="${joint_base_type}" parent="${base_parent}" child="${prefix}_link_base" joint_axis_xyz="${joint_base_axis_xyz}" joint_origin_xyz="${joint_base_origin_xyz}" joint_origin_rpy="${joint_base_origin_rpy}" joint_lower_limit="0" joint_upper_limit="0" fixed="true"/>
+        <!--xacro:kinova_armjoint joint_name="${prefix}_joint_base" type="${joint_base_type}" parent="${base_parent}" child="${prefix}_link_base" joint_axis_xyz="${joint_base_axis_xyz}" joint_origin_xyz="${joint_base_origin_xyz}" joint_origin_rpy="${joint_base_origin_rpy}" joint_lower_limit="0" joint_upper_limit="0" fixed="true"/> -->
+	 	<xacro:kinova_armjoint joint_name="${prefix}_joint_base" type="${joint_base_type}" parent="${base_parent}" child="${prefix}_link_base" joint_axis_xyz="${joint_base_axis_xyz}" joint_origin_xyz="${origin_xyz}" joint_origin_rpy="${origin_rpy}" joint_lower_limit="0" joint_upper_limit="0" fixed="true"/>
         <xacro:kinova_armlink link_name="${prefix}_link_1" link_mesh="${link_1_mesh}" use_ring_mesh="true" mesh_no="${link_1_mesh_no}"/>
         <xacro:kinova_armjoint joint_name="${prefix}_joint_1" type="${joint_1_type}" parent="${prefix}_link_base" child="${prefix}_link_1" joint_axis_xyz="${joint_1_axis_xyz}" joint_origin_xyz="${joint_1_origin_xyz}" joint_origin_rpy="${joint_1_origin_rpy}" joint_lower_limit="${joint_1_lower_limit}" joint_upper_limit="${joint_1_upper_limit}"/>
@@ -116,4 +118,7 @@
         <xacro:kinova_armlink link_name="${prefix}_link_6" link_mesh="${link_6_mesh}" use_ring_mesh="true" ring_mesh="ring_small" mesh_no="${link_6_mesh_no}"/>
         <xacro:kinova_armjoint joint_name="${prefix}_joint_6" type="${joint_6_type}" parent="${prefix}_link_5" child="${prefix}_link_6" joint_axis_xyz="${joint_6_axis_xyz}" joint_origin_xyz="${joint_6_origin_xyz}" joint_origin_rpy="${joint_6_origin_rpy}" joint_lower_limit="${joint_6_lower_limit}" joint_upper_limit="${joint_6_upper_limit}"/>
+		<!--xacro:kinova_armlink link_name="${prefix}_link_7"/> -->
+		<link name="${prefix}_link_7"/>
+		<xacro:kinova_armjoint joint_name="${prefix}_joint_7" type="${joint_7_type}" parent="${prefix}_link_6" child="${prefix}_link_7" joint_axis_xyz="${joint_7_axis_xyz}" joint_origin_xyz="${joint_7_origin_xyz}" joint_origin_rpy="${joint_7_origin_rpy}" joint_lower_limit="${joint_7_lower_limit}" joint_upper_limit="${joint_7_upper_limit}"/>
 <!--
         <xacro:kinova_armlink link_name="${prefix}_link_7" link_mesh="${link_7_mesh}" use_ring_mesh="true" ring_mesh="ring_small" mesh_no="${link_7_mesh_no}"/>

File: vector_common/vector_description/urdf/vector_7dof.urdf.xacro (robot description, xacro)
@@ -26,5 +26,5 @@
     <xacro:include filename="$(find vector_description)/urdf/linear_actuator/vector_linear_actuator.urdf.xacro" />
     <xacro:include filename="$(find vector_description)/urdf/accessories.urdf.xacro" />
-    <xacro:include filename="$(find kinova_description)/urdf/j2s7s300_mod.xacro" />
+    <xacro:include filename="$(find vector_description)/urdf/manipulation/jaco/j2s7s300_mod.xacro" />
     <xacro:include filename="$(find vector_description)/urdf/manipulation/robotiq/robotiq_85_gripper.urdf.xacro" />
     <xacro:property name="M_PI" value="3.14159"/>
@@ -81,5 +81,5 @@
     </xacro:if> -->
     <xacro:if value="$(optenv VECTOR_HAS_KINOVA_ARM false)">
-	<xacro:j2s7s300 prefix="right" base_parent="linear_actuator_link" origin_xyz="0.06079866 -0.1319 0" origin_rpy="${M_PI/2} 0 ${M_PI/2}" />
+		<xacro:j2s7s300 prefix="right" base_parent="linear_actuator_link" origin_xyz="0.06079866 -0.1319 0" origin_rpy="${M_PI/2} 0 ${M_PI/2}" />
         <!--<xacro:j2s7s300 prefix="right_" base_parent="linear_actuator_link">
             <xacro:unless value="$(optenv VECTOR_HAS_TWO_KINOVA_ARMS false)">
@@ -96,9 +96,9 @@
         </xacro:if>
         <xacro:if value="$(optenv VECTOR_HAS_ROBOTIQ_GRIPPER false)">
-            <xacro:robotiq_85_gripper prefix="right_" parent="right_link_6" >
+            <xacro:robotiq_85_gripper prefix="right_" parent="right_link_7" >
                 <origin xyz="0 0.10375 0" rpy="-${M_PI/2} 0 ${M_PI/2}"/>
             </xacro:robotiq_85_gripper>
             <xacro:if value="$(optenv VECTOR_HAS_TWO_ROBOTIQ_GRIPPERS false)">
-                <xacro:robotiq_85_gripper prefix="left_" parent="left_link_6" >
+                <xacro:robotiq_85_gripper prefix="left_" parent="left_link_7" >
                     <origin xyz="0 0.10375 0" rpy="-${M_PI/2} 0 ${M_PI/2}"/>
                 </xacro:robotiq_85_gripper>

Commit message: updated working urdf

File: vector_common/vector_description/urdf/manipulation/jaco/j2s7s300_mod.xacro (robot description, xacro)
@@ -15,7 +15,8 @@
     xmlns:xacro="http://ros.org/wiki/xacro">
     <xacro:include filename="$(find kinova_description)/urdf/kinova_common.xacro" />
+	<xacro:include filename="$(find vector_description)/urdf/manipulation/jaco/j2s7s300.transmission.xacro" />
     <!-- <xacro:include filename="$(find kinova_description)/urdf/kinova_finger_set.xacro" /> -->
     <!-- Import all Gazebo-customization elements -->
-    <xacro:include filename="$(find kinova_description)/urdf/kinova.gazebo" />
+    <!--<xacro:include filename="$(find kinova_description)/urdf/kinova.gazebo" /> -->
     <property name="link_base_mesh" value="base" />
     <property name="link_1_mesh" value="shoulder" />
@@ -128,4 +129,5 @@
         <xacro:kinova_virtual_joint joint_name="${prefix}_joint_end_effector" type="${joint_end_effector_type}" parent="${prefix}_link_7" child="${prefix}_end_effector" joint_axis_xyz="${joint_end_effector_axis_xyz}" joint_origin_xyz="${joint_end_effector_origin_xyz}" joint_origin_rpy="${joint_end_effector_origin_rpy}" joint_lower_limit="0" joint_upper_limit="0"/>
         <xacro:kinova_3fingers link_hand="${prefix}_link_7" prefix="${prefix}_"/> -->
+		<xacro:jaco_arm_transmission prefix="${prefix}" />
     </xacro:macro>
 </root>

File: vector_common/vector_description/urdf/vector_7dof.urdf.xacro (robot description, xacro)
@@ -97,9 +97,11 @@
         <xacro:if value="$(optenv VECTOR_HAS_ROBOTIQ_GRIPPER false)">
             <xacro:robotiq_85_gripper prefix="right_" parent="right_link_7" >
-                <origin xyz="0 0.10375 0" rpy="-${M_PI/2} 0 ${M_PI/2}"/>
+                <!-- <origin xyz="0 0.10375 0" rpy="-${M_PI/2} 0 ${M_PI/2}"/> -->
+				<origin xyz="0 0 0" rpy="0 ${M_PI/2} 0"/>
             </xacro:robotiq_85_gripper>
             <xacro:if value="$(optenv VECTOR_HAS_TWO_ROBOTIQ_GRIPPERS false)">
                 <xacro:robotiq_85_gripper prefix="left_" parent="left_link_7" >
-                    <origin xyz="0 0.10375 0" rpy="-${M_PI/2} 0 ${M_PI/2}"/>
+                    <!-- <origin xyz="0 0.10375 0" rpy="-${M_PI/2} 0 ${M_PI/2}"/> -->
+					<origin xyz="0 0 0" rpy="0 ${M_PI/2} 0"/>
                 </xacro:robotiq_85_gripper>
             </xacro:if>
