Commit message: Need to modify urdf

File: vector_common/vector_description/urdf/manipulation/jaco/j2s7s300.xacro (robot description, xacro)
@@ -95,4 +95,8 @@
     <property name="joint_7_lower_limit" value="${-2*J_PI}" />
     <property name="joint_7_upper_limit" value="${2*J_PI}" />
+    <property name="ee_fixed_joint" value="ee_fixed_joint" />
+    <property name="ee_fixed_joint_type" value="fixed" />
+    <property name="ee_fixed_joint_origin_xyz" value="0 0 -0.09380704" />
+    <property name="ee_fixed_joint_origin_rpy" value="${M_PI} ${M_PI/2} 0" />
 	<!--
     <property name="joint_end_effector" value="end_effector_offset" />
@@ -122,4 +126,20 @@
 		<link name="${prefix}_link_7"/>
 		<xacro:kinova_armjoint joint_name="${prefix}_joint_7" type="${joint_7_type}" parent="${prefix}_link_6" child="${prefix}_link_7" joint_axis_xyz="${joint_7_axis_xyz}" joint_origin_xyz="${joint_7_origin_xyz}" joint_origin_rpy="${joint_7_origin_rpy}" joint_lower_limit="${joint_7_lower_limit}" joint_upper_limit="${joint_7_upper_limit}"/>
+		<!-- -->
+		<!--xacro:kinova_armjoint joint_name="${prefix}_ee_fixed_joint" type="${ee_fixed_joint_type}" parent="${prefix}_link_7" child="${prefix}_ee_base" joint_origin_xyz="${joint_6_origin_xyz}" joint_origin_rpy="${joint_6_origin_rpy}"/-->
+		<joint name="${prefix}_ee_fixed_joint" type="fixed">
+            <parent link="${prefix}_link_7" />
+            <child link = "${prefix}_ee_base" />
+            <origin xyz="0 0 -0.09380704" rpy="${M_PI} ${M_PI/2} 0" /> <!--0.09380704156-->
+        </joint>
+        <link name="${prefix}_ee_base"/>
+        <!-- Add in an EEF link for the center of the gripper -->
+        <!--xacro:kinova_armjoint joint_name="${prefix}_ee_fixed_joint" type="fixed" parent="${prefix}_ee_base" child="${prefix}_ee_link" joint_origin_xyz="0.13 0 0"/-->
+        <joint name="${prefix}_ee_gripper" type="fixed">
+            <parent link="${prefix}_ee_base" />
+            <child link ="${prefix}_ee_link" />
+            <origin xyz="0.13 0 0" />
+        </joint>
+        <link name="${prefix}_ee_link"/>
 <!--
         <xacro:kinova_armlink link_name="${prefix}_link_7" link_mesh="${link_7_mesh}" use_ring_mesh="true" ring_mesh="ring_small" mesh_no="${link_7_mesh_no}"/>

Commit message: Updated urdf to add link 7

File: vector_common/vector_description/urdf/manipulation/jaco/j2s7s300.xacro (robot description, xacro)
@@ -26,5 +26,5 @@
     <property name="link_5_mesh" value="wrist_spherical_1" />
     <property name="link_6_mesh" value="wrist_spherical_2" />
-    <!-- <property name="link_7_mesh" value="hand_3finger" /> -->
+    <property name="link_7_mesh" value="wrist_3" />
     <!--Used for conditional arguments for setting inertial parameters
         base 0, shoulder 1, arm 2, forearm 3, wrist 4, arm_mico 5,
@@ -40,5 +40,6 @@
     <property name="link_5_mesh_no" value="8" />
     <property name="link_6_mesh_no" value="9" />
-    <!-- <property name="link_7_mesh_no" value="55" /> -->
+    <!-- <property name="link_7_mesh_no" value="11" /> -->
+    <property name="link_7_mesh_no" value="55" />
     <property name="joint_base" value="joint_base" />
     <property name="joint_base_type" value="fixed" />
@@ -91,12 +92,9 @@
     <property name="joint_7_type" value="continuous" />
     <property name="joint_7_axis_xyz" value="0 0 1" />
-    <property name="joint_7_origin_xyz" value="0 0.10375 0" />
+    <!--property name="joint_7_origin_xyz" value="0 0.10375 0" /-->
+    <property name="joint_7_origin_xyz" value="0 0.060 0" />
     <property name="joint_7_origin_rpy" value="${-J_PI/2} 0 ${J_PI}" />
     <property name="joint_7_lower_limit" value="${-2*J_PI}" />
     <property name="joint_7_upper_limit" value="${2*J_PI}" />
-    <property name="ee_fixed_joint" value="ee_fixed_joint" />
-    <property name="ee_fixed_joint_type" value="fixed" />
-    <property name="ee_fixed_joint_origin_xyz" value="0 0 -0.09380704" />
-    <property name="ee_fixed_joint_origin_rpy" value="${M_PI} ${M_PI/2} 0" />
 	<!--
     <property name="joint_end_effector" value="end_effector_offset" />
@@ -107,5 +105,5 @@
     <xacro:macro name="j2s7s300" params="base_parent prefix origin_xyz origin_rpy">
         <!--xacro:gazebo_config robot_namespace="${prefix}"/> -->
-        <xacro:gazebo_config robot_namespace="/"/>
+        <!-- <xacro:gazebo_config robot_namespace="/"/> -->
         <xacro:kinova_armlink link_name="${prefix}_link_base" link_mesh="${link_base_mesh}" mesh_no="${link_base_mesh_no}"/>
         <!--xacro:kinova_armjoint joint_name="${prefix}_joint_base" type="${joint_base_type}" parent="${base_parent}" child="${prefix}_link_base" joint_axis_xyz="${joint_base_axis_xyz}" joint_origin_xyz="${joint_base_origin_xyz}" joint_origin_rpy="${joint_base_origin_rpy}" joint_lower_limit="0" joint_upper_limit="0" fixed="true"/> -->
@@ -124,9 +122,10 @@
         <xacro:kinova_armjoint joint_name="${prefix}_joint_6" type="${joint_6_type}" parent="${prefix}_link_5" child="${prefix}_link_6" joint_axis_xyz="${joint_6_axis_xyz}" joint_origin_xyz="${joint_6_origin_xyz}" joint_origin_rpy="${joint_6_origin_rpy}" joint_lower_limit="${joint_6_lower_limit}" joint_upper_limit="${joint_6_upper_limit}"/>
 		<!--xacro:kinova_armlink link_name="${prefix}_link_7"/> -->
-		<link name="${prefix}_link_7"/>
-		<xacro:kinova_armjoint joint_name="${prefix}_joint_7" type="${joint_7_type}" parent="${prefix}_link_6" child="${prefix}_link_7" joint_axis_xyz="${joint_7_axis_xyz}" joint_origin_xyz="${joint_7_origin_xyz}" joint_origin_rpy="${joint_7_origin_rpy}" joint_lower_limit="${joint_7_lower_limit}" joint_upper_limit="${joint_7_upper_limit}"/>
-		<!-- -->
-		<!--xacro:kinova_armjoint joint_name="${prefix}_ee_fixed_joint" type="${ee_fixed_joint_type}" parent="${prefix}_link_7" child="${prefix}_ee_base" joint_origin_xyz="${joint_6_origin_xyz}" joint_origin_rpy="${joint_6_origin_rpy}"/-->
-		<joint name="${prefix}_ee_fixed_joint" type="fixed">
+		<!--link name="${prefix}_link_7"/-->
+<!-- 		<xacro:kinova_armjoint joint_name="${prefix}_joint_7" type="${joint_7_type}" parent="${prefix}_link_6" child="${prefix}_link_7" joint_axis_xyz="${joint_7_axis_xyz}" joint_origin_xyz="${joint_7_origin_xyz}" joint_origin_rpy="${joint_7_origin_rpy}" joint_lower_limit="${joint_7_lower_limit}" joint_upper_limit="${joint_7_upper_limit}"/> -->
+	   <!-- Modifications to mount robotiq gripper -->
+        <xacro:kinova_armlink link_name="${prefix}_link_7" link_mesh="${link_7_mesh}" use_ring_mesh="false" ring_mesh="ring_small" mesh_no="${link_7_mesh_no}"/>
+        <xacro:kinova_armjoint joint_name="${prefix}_joint_7" type="${joint_7_type}" parent="${prefix}_link_6" child="${prefix}_link_7" joint_axis_xyz="${joint_7_axis_xyz}" joint_origin_xyz="${joint_7_origin_xyz}" joint_origin_rpy="${joint_7_origin_rpy}" joint_lower_limit="${joint_7_lower_limit}" joint_upper_limit="${joint_7_upper_limit}"/>
+        <joint name="${prefix}_ee_fixed_joint" type="fixed">
             <parent link="${prefix}_link_7" />
             <child link = "${prefix}_ee_base" />
@@ -135,5 +134,4 @@
         <link name="${prefix}_ee_base"/>
         <!-- Add in an EEF link for the center of the gripper -->
-        <!--xacro:kinova_armjoint joint_name="${prefix}_ee_fixed_joint" type="fixed" parent="${prefix}_ee_base" child="${prefix}_ee_link" joint_origin_xyz="0.13 0 0"/-->
         <joint name="${prefix}_ee_gripper" type="fixed">
             <parent link="${prefix}_ee_base" />

File: vector_common/vector_description/urdf/vector_7dof.urdf.xacro (robot description, xacro)
@@ -94,12 +94,14 @@
             <xacro:j2s7s300 prefix="left" base_parent="linear_actuator_link" origin_xyz="0.06079866 0.1319 0" origin_rpy="${M_PI/2} 0 ${M_PI/2}" />
         <xacro:if value="$(optenv VECTOR_HAS_ROBOTIQ_GRIPPER false)">
-            <xacro:robotiq_85_gripper prefix="right_" parent="right_link_7" >
+            <!-- <xacro:robotiq_85_gripper prefix="right_" parent="right_link_7" > -->
+            <xacro:robotiq_85_gripper prefix="right_" parent="right_ee_base" >
                 <!-- <origin xyz="0 0.10375 0" rpy="-${M_PI/2} 0 ${M_PI/2}"/> -->
-				<origin xyz="0 0 0" rpy="0 ${M_PI/2} 0"/>
+				<origin xyz="0 0 0" rpy="0 0 0"/>
             </xacro:robotiq_85_gripper>
             <xacro:if value="$(optenv VECTOR_HAS_TWO_ROBOTIQ_GRIPPERS false)">
-                <xacro:robotiq_85_gripper prefix="left_" parent="left_link_7" >
+                <!-- <xacro:robotiq_85_gripper prefix="left_" parent="left_link_7" > -->
+                <xacro:robotiq_85_gripper prefix="left_" parent="left_ee_base" >
                     <!-- <origin xyz="0 0.10375 0" rpy="-${M_PI/2} 0 ${M_PI/2}"/> -->
-					<origin xyz="0 0 0" rpy="0 ${M_PI/2} 0"/>
+					<origin xyz="0 0 0" rpy="0 0 0"/>
                 </xacro:robotiq_85_gripper>
             </xacro:if>

Commit message: Updated urdf to have correct tf tree

File: vector_common/vector_description/urdf/manipulation/jaco/j2s7s300.xacro (robot description, xacro)
@@ -94,4 +94,5 @@
     <!--property name="joint_7_origin_xyz" value="0 0.10375 0" /-->
     <property name="joint_7_origin_xyz" value="0 0.060 0" />
+    <!--property name="joint_7_origin_xyz" value="0 0 0" /-->
     <property name="joint_7_origin_rpy" value="${-J_PI/2} 0 ${J_PI}" />
     <property name="joint_7_lower_limit" value="${-2*J_PI}" />
@@ -130,5 +131,6 @@
             <parent link="${prefix}_link_7" />
             <child link = "${prefix}_ee_base" />
-            <origin xyz="0 0 -0.09380704" rpy="${M_PI} ${M_PI/2} 0" /> <!--0.09380704156-->
+            <origin xyz="0 0 -0.09380704" rpy="${M_PI/2} ${M_PI/2} 0" /> <!--0.09380704156-->
+            <!--origin xyz="0 0 -0.09380704" rpy="0 ${M_PI/2} 0" /-->
         </joint>
         <link name="${prefix}_ee_base"/>
