Commit message: updating gazebo collision and inertial properties to fix simulation

File: vector_common/vector_description/urdf/vector_components/vector_base.urdf.xacro (robot description, xacro)
@@ -34,9 +34,9 @@
         <link name="${name}_chassis_link">
 			<inertial>
-				<mass value="36.914402" />
-				<origin xyz="-0.043407 0.000037 0.060079" />
-				<inertia ixx="1.182744"  ixy="0.017957" ixz="-0.077476"
-                         iyx="0.017957"  iyy="0.538664" iyz="0.000018"
-                         izx="-0.077476" izy="0.000018" izz="1.240229" />
+				<mass value="55.914402" />
+				<origin xyz="0 0 0" />
+				<inertia ixx="3.54"  ixy="0" ixz="0"
+                         iyx="0"  iyy="3.71" iyz="0"
+                         izx="0" izy="0" izz="2.53" />
 			</inertial>
             <collision>
@@ -52,4 +52,12 @@
 			</visual>
 		</link>
+		<gazebo reference="${name}_chassis_link">
+			<mu1 value="100.0"/>
+			<mu2 value="100.0"/>
+			<kp value="10000000.0" />
+			<kd value="10.0" />
+			<fdir1 value="1 0 0"/>
+			<minDepth>0.003</minDepth>
+		</gazebo>
     </xacro:macro>
 </robot>

Commit message: initial trial, need to debug simulator

File: vector_common/vector_description/urdf/vector_components/vector_base.urdf.xacro (robot description, xacro)
@@ -36,11 +36,19 @@
         </joint>
         <link name="${name}_chassis_link">
-			<inertial>
-				<mass value="55.914402" />
-				<origin xyz="0 0 0" />
-				<inertia ixx="3.54"  ixy="0" ixz="0"
-                         iyx="0"  iyy="3.71" iyz="0"
-                         izx="0" izy="0" izz="2.53" />
-			</inertial>
+            <inertial>
+                <mass value="55.914402" />
+                <origin xyz="0 0 0" />
+                <xacro:unless value="$(arg simulation_urdf)">
+                    <inertia ixx="3.53"  ixy="0" ixz="0"
+                             iyx="0"  iyy="3.71" iyz="0"
+                             izx="0" izy="0" izz="2.53" />
+                </xacro:unless>
+                <!-- Set appropriate inertial values if in simulation -->
+                <xacro:if value="$(arg simulation_urdf)">
+                    <inertia ixx="3000"  ixy="0" ixz="0"
+                             iyx="3000"  iyy="3.71" iyz="0"
+                             izx="3000" izy="0" izz="2.53" />
+                </xacro:if>
+            </inertial>
             <collision>
 				<geometry>
